Commit message: Update

File: src/baxter_description/urdf/baxter.urdf.xacro (robot description, xacro)
@@ -3,13 +3,12 @@
   <xacro:arg name="gazebo" default="false"/>
   <xacro:arg name="pedestal" default="true"/>
-  <xacro:property name="PI" value="3.1415927"/>
   <!-- Baxter Base URDF -->
   <xacro:include filename="$(find baxter_description)/urdf/baxter_base/baxter_base.urdf.xacro">
-<!--     <xacro:arg name="gazebo" value="$(arg gazebo)"/> -->
+    <xacro:arg name="gazebo" value="${gazebo}"/>
   </xacro:include>
   <!-- Baxter Pedestal -->
   <xacro:if value="$(arg pedestal)">
     <xacro:include filename="$(find baxter_description)/urdf/pedestal/pedestal.xacro">
-<!--       <xacro:arg name="gazebo" value="$(arg gazebo)"/> -->
+      <xacro:arg name="gazebo" value="${gazebo}"/>
     </xacro:include>
   </xacro:if>
@@ -18,5 +17,3 @@
   <!-- Right End Effector -->
   <xacro:include filename="$(find baxter_description)/urdf/right_end_effector.urdf.xacro" />
-  <!-- Gazebo plugins -->
-  <xacro:include filename="$(find baxter_description)/urdf/gazebosim.urdf.xacro" />
 </robot>

File: src/baxter_description/urdf/baxter_base/baxter_base.urdf.xacro (robot description, xacro)
@@ -1,43 +1,9 @@
 <?xml version="1.0" ?>
 <robot name="baxter" xmlns:xacro="http://www.ros.org/wiki/xacro">
-<!--  <xacro:if value="$(arg gazebo)">
-    <xacro:property name="mass_scale" value=".1"/>
+  <xacro:arg name="gazebo" default="false"/>
+  <xacro:if value="$(arg gazebo)">
+    <!-- Gazebo Tags -->
     <xacro:include filename="$(find baxter_description)/urdf/baxter_base/baxter_base.gazebo.xacro" />
   </xacro:if>
-  <xacro:unless value="$(arg gazebo)">
-    <xacro:property name="mass_scale" value=".1"/>
-  </xacro:unless>-->
-  <xacro:macro name="range_sensor" params="side">
- <!-- <gazebo>
-  <sensor name="range_${side}" type="gpu_lidar">
-    <pose >1 0 0 0 ${PI/2} 0</pose>
-    <topic>${side}_range</topic>
-    <update_rate>10</update_rate>
-    <ray>
-        <scan>
-<horizontal>
-                <samples>10</samples>
-                <resolution>1</resolution>
-                <min_angle>-1.396263</min_angle>
-                <max_angle>1.396263</max_angle>
-            </horizontal>
-            <vertical>
-                <samples>1</samples>
-                <resolution>0.01</resolution>
-                <min_angle>0</min_angle>
-                <max_angle>0</max_angle>
-            </vertical>
-        </scan>
-        <range>
-            <min>0.1</min>
-            <max>1.</max>
-            <resolution>0.01</resolution>
-        </range>
-    </ray>
-    <always_on>1</always_on>
-    <visualize>true</visualize>
-</sensor>
-</gazebo>-->
-</xacro:macro>
   <link name="base">
   </link>
@@ -46,5 +12,5 @@
       <origin rpy="0 0 0" xyz="0 0 0"/>
       <geometry>
-        <mesh filename="file://$(find baxter_description)/meshes/torso/base_link.DAE"/>
+        <mesh filename="package://baxter_description/meshes/torso/base_link.DAE"/>
       </geometry>
       <material name="darkgray">
@@ -55,5 +21,5 @@
       <origin rpy="0 0 0" xyz="0 0 0"/>
       <geometry>
-        <mesh filename="file://$(find baxter_description)/meshes/torso/base_link_collision.DAE"/>
+        <mesh filename="package://baxter_description/meshes/torso/base_link_collision.DAE"/>
       </geometry>
     </collision>
@@ -82,5 +48,5 @@
       <origin rpy="0 0 0" xyz="0 0 .00953"/>
       <geometry>
-        <mesh filename="file://$(find baxter_description)/meshes/head/H0.DAE"/>
+        <mesh filename="package://baxter_description/meshes/head/H0.DAE"/>
       </geometry>
       <material name="darkgray">
@@ -126,5 +92,5 @@
       <origin rpy="0 -1.57079632679 0" xyz="0 -.00953 -.0347"/>
       <geometry>
-        <mesh filename="file://$(find baxter_description)/meshes/head/H1.DAE"/>
+        <mesh filename="package://baxter_description/meshes/head/H1.DAE"/>
       </geometry>
       <material name="darkred">
@@ -262,5 +228,5 @@
     <child link="screen"/>
   </joint>
-  <joint name="head_camera_fixed" type="fixed">
+  <joint name="head_camera" type="fixed">
     <origin rpy="1.75057 0 1.57079632679" xyz="0.12839 0 0.06368"/>
     <parent link="head"/>
@@ -290,5 +256,5 @@
       <origin rpy="0 0 0" xyz="0 0 0"/>
       <geometry>
-        <mesh filename="file://$(find baxter_description)/meshes/upper_shoulder/S0.DAE"/>
+        <mesh filename="package://baxter_description/meshes/upper_shoulder/S0.DAE"/>
       </geometry>
       <material name="darkred">
@@ -312,5 +278,5 @@
       <origin rpy="0 0 0" xyz="0 0 0"/>
       <geometry>
-        <mesh filename="file://$(find baxter_description)/meshes/lower_shoulder/S1.DAE"/>
+        <mesh filename="package://baxter_description/meshes/lower_shoulder/S1.DAE"/>
       </geometry>
       <material name="darkred">
@@ -334,5 +300,5 @@
       <origin rpy="0 0 0" xyz="0 0 0"/>
       <geometry>
-        <mesh filename="file://$(find baxter_description)/meshes/upper_elbow/E0.DAE"/>
+        <mesh filename="package://baxter_description/meshes/upper_elbow/E0.DAE"/>
       </geometry>
       <material name="darkred">
@@ -369,5 +335,5 @@
       <origin rpy="0 0 0" xyz="0 0 0"/>
       <geometry>
-        <mesh filename="file://$(find baxter_description)/meshes/lower_elbow/E1.DAE"/>
+        <mesh filename="package://baxter_description/meshes/lower_elbow/E1.DAE"/>
       </geometry>
       <material name="darkred">
@@ -391,5 +357,5 @@
       <origin rpy="0 0 0" xyz="0 0 0"/>
       <geometry>
-        <mesh filename="file://$(find baxter_description)/meshes/upper_forearm/W0.DAE"/>
+        <mesh filename="package://baxter_description/meshes/upper_forearm/W0.DAE"/>
       </geometry>
       <material name="darkred">
@@ -433,5 +399,5 @@
       <origin rpy="0 0 0" xyz="0 0 0"/>
       <geometry>
-        <mesh filename="file://$(find baxter_description)/meshes/lower_forearm/W1.DAE"/>
+        <mesh filename="package://baxter_description/meshes/lower_forearm/W1.DAE"/>
       </geometry>
       <material name="darkred">
@@ -455,5 +421,5 @@
       <origin rpy="0 0 0" xyz="0 0 0"/>
       <geometry>
-        <mesh filename="file://$(find baxter_description)/meshes/wrist/W2.DAE"/>
+        <mesh filename="package://baxter_description/meshes/wrist/W2.DAE"/>
       </geometry>
       <material name="lightgrey">
@@ -524,5 +490,4 @@
       <inertia ixx="1e-08" ixy="0" ixz="0" iyy="1e-08" iyz="0" izz="1e-08"/>
     </inertial>
-    <xacro:range_sensor side="right"/>
   </link>
   <link name="right_hand_accelerometer">
@@ -621,5 +586,5 @@
     <dynamics damping="0.7" friction="0.0"/>
   </joint>
-  <joint name="right_hand_fixed" type="fixed">
+  <joint name="right_hand" type="fixed">
     <origin rpy="0 0 0" xyz="0 0 0.11355"/>
     <axis xyz="0 0 1"/>
@@ -627,20 +592,20 @@
     <child link="right_hand"/>
   </joint>
-  <joint name="right_hand_camera_fixed" type="fixed">
+  <joint name="right_hand_camera" type="fixed">
     <origin rpy="0 0 -1.57079633" xyz="0.03825 0.012 0.015355"/>
     <parent link="right_hand"/>
     <child link="right_hand_camera"/>
   </joint>
-  <joint name="right_hand_camera_axis_fixed" type="fixed">
+  <joint name="right_hand_camera_axis" type="fixed">
     <origin rpy="0 0 0" xyz="0.03825 0.012 0.015355"/>
     <parent link="right_hand"/>
     <child link="right_hand_camera_axis"/>
   </joint>
-  <joint name="right_hand_range_fixed" type="fixed">
+  <joint name="right_hand_range" type="fixed">
     <origin rpy="0 -1.57079632679 -1.57079632679" xyz="0.032 -0.020245 0.0288"/>
     <parent link="right_hand"/>
     <child link="right_hand_range"/>
   </joint>
-  <joint name="right_hand_accelerometer_fixed" type="fixed">
+  <joint name="right_hand_accelerometer" type="fixed">
     <origin rpy="0 0 0" xyz="0.00198 0.000133 -0.0146"/>
     <parent link="right_hand"/>
@@ -659,5 +624,5 @@
       <origin rpy="0 0 0" xyz="0 0 0"/>
       <geometry>
-        <mesh filename="file://$(find baxter_description)/meshes/upper_shoulder/S0.DAE"/>
+        <mesh filename="package://baxter_description/meshes/upper_shoulder/S0.DAE"/>
       </geometry>
       <material name="darkred">
@@ -681,5 +646,5 @@
       <origin rpy="0 0 0" xyz="0 0 0"/>
       <geometry>
-        <mesh filename="file://$(find baxter_description)/meshes/lower_shoulder/S1.DAE"/>
+        <mesh filename="package://baxter_description/meshes/lower_shoulder/S1.DAE"/>
       </geometry>
       <material name="darkred">
@@ -703,5 +668,5 @@
       <origin rpy="0 0 0" xyz="0 0 0"/>
       <geometry>
-        <mesh filename="file://$(find baxter_description)/meshes/upper_elbow/E0.DAE"/>
+        <mesh filename="package://baxter_description/meshes/upper_elbow/E0.DAE"/>
       </geometry>
       <material name="darkred">
@@ -738,5 +703,5 @@
       <origin rpy="0 0 0" xyz="0 0 0"/>
       <geometry>
-        <mesh filename="file://$(find baxter_description)/meshes/lower_elbow/E1.DAE"/>
+        <mesh filename="package://baxter_description/meshes/lower_elbow/E1.DAE"/>
       </geometry>
       <material name="darkred">
@@ -760,5 +725,5 @@
       <origin rpy="0 0 0" xyz="0 0 0"/>
       <geometry>
-        <mesh filename="file://$(find baxter_description)/meshes/upper_forearm/W0.DAE"/>
+        <mesh filename="package://baxter_description/meshes/upper_forearm/W0.DAE"/>
       </geometry>
       <material name="darkred">
@@ -802,5 +767,5 @@
       <origin rpy="0 0 0" xyz="0 0 0"/>
       <geometry>
-        <mesh filename="file://$(find baxter_description)/meshes/lower_forearm/W1.DAE"/>
+        <mesh filename="package://baxter_description/meshes/lower_forearm/W1.DAE"/>
       </geometry>
       <material name="darkred">
@@ -824,5 +789,5 @@
       <origin rpy="0 0 0" xyz="0 0 0"/>
       <geometry>
-        <mesh filename="file://$(find baxter_description)/meshes/wrist/W2.DAE"/>
+        <mesh filename="package://baxter_description/meshes/wrist/W2.DAE"/>
       </geometry>
       <material name="lightgrey">
@@ -909,5 +874,4 @@
       <inertia ixx="1e-08" ixy="0" ixz="0" iyy="1e-08" iyz="0" izz="1e-08"/>
     </inertial>
-    <xacro:range_sensor side="left"/>
   </link>
   <joint name="left_torso_arm_mount" type="fixed">
@@ -990,5 +954,5 @@
     <dynamics damping="0.7" friction="0.0"/>
   </joint>
-  <joint name="left_hand_fixed" type="fixed">
+  <joint name="left_hand" type="fixed">
     <origin rpy="0 0 0" xyz="0 0 0.11355"/>
     <axis xyz="0 0 1"/>
@@ -996,20 +960,20 @@
     <child link="left_hand"/>
   </joint>
-  <joint name="left_hand_camera_fixed" type="fixed">
+  <joint name="left_hand_camera" type="fixed">
     <origin rpy="0 0 -1.57079633" xyz="0.03825 0.012 0.015355"/>
     <parent link="left_hand"/>
     <child link="left_hand_camera"/>
   </joint>
-  <joint name="left_hand_camera_axis_fixed" type="fixed">
+  <joint name="left_hand_camera_axis" type="fixed">
     <origin rpy="0 0 0" xyz="0.03825 0.012 0.015355"/>
     <parent link="left_hand"/>
     <child link="left_hand_camera_axis"/>
   </joint>
-  <joint name="left_hand_range_fixed" type="fixed">
+  <joint name="left_hand_range" type="fixed">
     <origin rpy="0 -1.57079632679 -1.57079632679" xyz="0.032 -0.020245 0.0288"/>
     <parent link="left_hand"/>
     <child link="left_hand_range"/>
   </joint>
-  <joint name="left_hand_accelerometer_fixed" type="fixed">
+  <joint name="left_hand_accelerometer" type="fixed">
     <origin rpy="0 0 0" xyz="0.00198 0.000133 -0.0146"/>
     <parent link="left_hand"/>

File: src/baxter_description/urdf/pedestal/pedestal.xacro (robot description, xacro)
@@ -1,11 +1,11 @@
 <?xml version="1.0" ?>
-<robot name="pedestal" xmlns:xacro="http://www.ros.org/wiki/xacro">
+<robot name="pedistal" xmlns:xacro="http://www.ros.org/wiki/xacro">
   <!-- Arguments and Defaults-->
-<!--   <xacro:arg name="gazebo" default="false"/> -->
+  <xacro:arg name="gazebo" default="false"/>
   <link name="pedestal">
     <visual>
       <origin rpy="0 0 0" xyz="0 0 0"/>
       <geometry>
-        <mesh filename="file://$(find baxter_description)/meshes/base/PEDESTAL.DAE"/>
+        <mesh filename="package://baxter_description/meshes/base/PEDESTAL.DAE"/>
       </geometry>
       <material name="darkgray">
@@ -16,5 +16,5 @@
       <origin rpy="0 0 0" xyz="0 0 0"/>
       <geometry>
-        <mesh filename="file://$(find baxter_description)/meshes/base/pedestal_link_collision.DAE"/>
+        <mesh filename="package://baxter_description/meshes/base/pedestal_link_collision.DAE"/>
       </geometry>
     </collision>
@@ -30,5 +30,6 @@
     <child link="pedestal"/>
   </joint>
-  <!--<xacro:if value="$(arg gazebo)">
+  <xacro:if value="$(arg gazebo)">
+    <!-- When using the pedistal, fix Baxter to Gazebo world with 'base' frame -->
     <link name="world"/>
     <joint name="fixed" type="fixed">
@@ -36,4 +37,4 @@
       <child link="base"/>
     </joint>
-  </xacro:if>-->
+  </xacro:if>
 </robot>
