Commit message: added baxter xacro spawn

File: src/baxter_description/urdf/left_end_effector.urdf.xacro (robot description, xacro)
@@ -1,13 +1,14 @@
-<?xml version="1.0" ?>
+<?xml version="1.0"?>
 <robot name="left_end_effector" xmlns:xacro="http://www.ros.org/wiki/xacro">
-  <xacro:include filename="$(find rethink_ee_description)/urdf/electric_gripper/rethink_electric_gripper.xacro" />
+  <xacro:include
+    filename="$(find rethink_ee_description)/urdf/electric_gripper/rethink_electric_gripper.xacro" />
   <xacro:rethink_electric_gripper side="left"
-                                  l_finger="extended_narrow"
-                                  l_finger_slot="2"
-                                  l_finger_tip="paddle_tip"
-                                  l_finger_grasp="inner"
-                                  r_finger="extended_narrow"
-                                  r_finger_slot="2"
-                                  r_finger_tip="paddle_tip"
-                                  r_finger_grasp="inner"/>
+    l_finger="extended_narrow"
+    l_finger_slot="2"
+    l_finger_tip="paddle_tip"
+    l_finger_grasp="inner"
+    r_finger="extended_narrow"
+    r_finger_slot="2"
+    r_finger_tip="paddle_tip"
+    r_finger_grasp="inner" />
 </robot>

File: src/baxter_description/urdf/right_end_effector.urdf.xacro (robot description, xacro)
@@ -1,13 +1,14 @@
-<?xml version="1.0" ?>
+<?xml version="1.0"?>
 <robot name="right_end_effector" xmlns:xacro="http://www.ros.org/wiki/xacro">
-  <xacro:include filename="$(find rethink_ee_description)/urdf/electric_gripper/rethink_electric_gripper.xacro" />
+  <xacro:include
+    filename="$(find rethink_ee_description)/urdf/electric_gripper/rethink_electric_gripper.xacro" />
   <xacro:rethink_electric_gripper side="right"
-                                  l_finger="extended_narrow"
-                                  l_finger_slot="2"
-                                  l_finger_tip="half_round_tip"
-                                  l_finger_grasp="inner"
-                                  r_finger="extended_narrow"
-                                  r_finger_slot="2"
-                                  r_finger_tip="half_round_tip"
-                                  r_finger_grasp="inner"/>
+    l_finger="extended_narrow"
+    l_finger_slot="2"
+    l_finger_tip="paddle_tip"
+    l_finger_grasp="inner"
+    r_finger="extended_narrow"
+    r_finger_slot="2"
+    r_finger_tip="paddle_tip"
+    r_finger_grasp="inner" />
 </robot>

File: src/rethink_ee_description/urdf/electric_gripper/fingers/basic_hard_tip.xacro (robot description, xacro)
@@ -10,5 +10,5 @@
         <origin rpy="0 0 ${pi*(g_reflect+1)/2}" xyz="0 0 0"/>
         <geometry>
-          <mesh filename="file://$(find rethink_ee_description)/meshes/electric_gripper/fingers/basic_hard_tip.DAE" />
+          <mesh filename="$(find rethink_ee_description)/meshes/electric_gripper/fingers/basic_hard_tip.DAE" />
         </geometry>
       </visual>

File: src/rethink_ee_description/urdf/electric_gripper/fingers/basic_soft_tip.xacro (robot description, xacro)
@@ -10,5 +10,5 @@
         <origin rpy="0 0 ${pi*(g_reflect+1)/2}" xyz="0 0 0"/>
         <geometry>
-          <mesh filename="file://$(find rethink_ee_description)/meshes/electric_gripper/fingers/basic_soft_tip.DAE" />
+          <mesh filename="$(find rethink_ee_description)/meshes/electric_gripper/fingers/basic_soft_tip.DAE" />
         </geometry>
       </visual>

File: src/rethink_ee_description/urdf/electric_gripper/fingers/extended_narrow.xacro (robot description, xacro)
@@ -8,5 +8,5 @@
         <origin rpy="0 0 ${-pi/2*(reflect+1)}" xyz="0 0 0"/>
         <geometry>
-          <mesh filename="file://$(find rethink_ee_description)/meshes/electric_gripper/fingers/extended_narrow.DAE" />
+          <mesh filename="$(find rethink_ee_description)/meshes/electric_gripper/fingers/extended_narrow.DAE" />
         </geometry>
       </visual>

File: src/rethink_ee_description/urdf/electric_gripper/fingers/extended_wide.xacro (robot description, xacro)
@@ -8,5 +8,5 @@
         <origin rpy="0 0 ${-pi/2*(reflect+1)}" xyz="0 0 0"/>
         <geometry>
-          <mesh filename="file://$(find rethink_ee_description)/meshes/electric_gripper/fingers/extended_wide.DAE" />
+          <mesh filename="$(find rethink_ee_description)/meshes/electric_gripper/fingers/extended_wide.DAE" />
         </geometry>
       </visual>

File: src/rethink_ee_description/urdf/electric_gripper/fingers/half_round_tip.xacro (robot description, xacro)
@@ -10,5 +10,5 @@
         <origin rpy="0 0 ${pi*(g_reflect+1)/2}" xyz="0 0 0"/>
         <geometry>
-          <mesh filename="file://$(find rethink_ee_description)/meshes/electric_gripper/fingers/half_round_tip.DAE" />
+          <mesh filename="$(find rethink_ee_description)/meshes/electric_gripper/fingers/half_round_tip.DAE" />
         </geometry>
       </visual>

File: src/rethink_ee_description/urdf/electric_gripper/fingers/paddle_tip.xacro (robot description, xacro)
@@ -10,5 +10,5 @@
         <origin rpy="0 0 ${pi*(g_reflect+1)/2}" xyz="0 0 0"/>
         <geometry>
-          <mesh filename="file://$(find rethink_ee_description)/meshes/electric_gripper/fingers/paddle_tip.DAE" />
+          <mesh filename="$(find rethink_ee_description)/meshes/electric_gripper/fingers/paddle_tip.DAE" />
         </geometry>
       </visual>

File: src/rethink_ee_description/urdf/electric_gripper/fingers/standard_narrow.xacro (robot description, xacro)
@@ -8,5 +8,5 @@
         <origin rpy="0 0 ${-pi/2*(reflect+1)}" xyz="0 0 0"/>
         <geometry>
-          <mesh filename="file://$(find rethink_ee_description)/meshes/electric_gripper/fingers/standard_narrow.DAE" />
+          <mesh filename="$(find rethink_ee_description)/meshes/electric_gripper/fingers/standard_narrow.DAE" />
         </geometry>
       </visual>

File: src/rethink_ee_description/urdf/electric_gripper/fingers/standard_wide.xacro (robot description, xacro)
@@ -8,5 +8,5 @@
         <origin rpy="0 0 ${-pi/2*(reflect+1)}" xyz="0 0 0"/>
         <geometry>
-          <mesh filename="file://$(find rethink_ee_description)/meshes/electric_gripper/fingers/standard_wide.DAE" />
+          <mesh filename="$(find rethink_ee_description)/meshes/electric_gripper/fingers/standard_wide.DAE" />
         </geometry>
       </visual>

File: src/rethink_ee_description/urdf/electric_gripper/rethink_electric_gripper.xacro (robot description, xacro)
@@ -1,80 +1,88 @@
 <?xml version="1.0"?>
 <robot xmlns:xacro="http://www.ros.org/wiki/xacro" name="rethink_electric_gripper">
-  <xacro:macro name="rethink_electric_gripper" params="side r_finger r_finger_slot r_finger_tip r_finger_grasp l_finger l_finger_slot l_finger_tip l_finger_grasp">
-    <xacro:property name="gripper_side" value="${side[0]}" scope="local"/>
+  <xacro:macro name="rethink_electric_gripper"
+    params="side r_finger r_finger_slot r_finger_tip r_finger_grasp l_finger l_finger_slot l_finger_tip l_finger_grasp">
+    <xacro:property name="gripper_side" value="${side[0]}" scope="local" />
     <!-- Base of end effector -->
     <link name="${side}_gripper_base">
       <visual>
-        <origin rpy="${-pi/2} ${pi} 0" xyz="0 0 0"/>
+        <origin rpy="${-pi/2} ${pi} 0" xyz="0 0 0" />
         <geometry>
-          <mesh filename="file://$(find rethink_ee_description)/meshes/electric_gripper/electric_gripper_base.DAE"/>
+          <mesh
+            filename="$(find rethink_ee_description)/meshes/electric_gripper/electric_gripper_base.DAE" />
         </geometry>
       </visual>
       <collision>
-        <origin rpy="${-pi/2} ${pi} 0" xyz="0.0 0.0 0"/>
+        <origin rpy="${-pi/2} ${pi} 0" xyz="0.0 0.0 0" />
         <geometry>
-          <cylinder length="0.1" radius="0.029"/>
+          <cylinder length="0.1" radius="0.029" />
         </geometry>
         <material name="darkred">
-          <color rgba=".5 .1 .1 1"/>
+          <color rgba=".5 .1 .1 1" />
         </material>
       </collision>
       <inertial>
-        <origin rpy="${-pi/2} ${pi} 0" xyz="0.0 0.0 0.0"/>
-        <mass value="0.3"/>
-        <inertia ixx="2e-08" ixy="0" ixz="0" iyy="3e-08" iyz="0" izz="2e-08"/>
+        <origin rpy="${-pi/2} ${pi} 0" xyz="0.0 0.0 0.0" />
+        <mass value="0.3" />
+        <inertia ixx="2e-08" ixy="0" ixz="0" iyy="3e-08" iyz="0" izz="2e-08" />
       </inertial>
     </link>
     <!-- Left finger link -->
-    <xacro:property name="finger_length" value="0.0" scope="global"/>
-    <xacro:include filename="$(find rethink_ee_description)/urdf/electric_gripper/fingers/${l_finger}.xacro" />
-    <xacro:finger_xacro gripper_side="${gripper_side}" finger_side="l" reflect="1" finger_tip="${l_finger_tip}" finger_grasp="${l_finger_grasp}"/>
-    <xacro:property name="tip_finger_length" value="${finger_length}" scope="local"/>
+    <xacro:property name="finger_length" value="0.0" scope="global" />
+    <xacro:include
+      filename="$(find rethink_ee_description)/urdf/electric_gripper/fingers/${l_finger}.xacro" />
+    <xacro:finger_xacro gripper_side="${gripper_side}" finger_side="l" reflect="1"
+      finger_tip="${l_finger_tip}" finger_grasp="${l_finger_grasp}" />
+    <xacro:property name="tip_finger_length" value="${finger_length}" scope="local" />
     <!-- Right finger link -->
-    <xacro:include filename="$(find rethink_ee_description)/urdf/electric_gripper/fingers/${r_finger}.xacro" />
-    <xacro:finger_xacro gripper_side="${gripper_side}" finger_side="r" reflect="-1" finger_tip="${r_finger_tip}" finger_grasp="${r_finger_grasp}"/>
+    <xacro:include
+      filename="$(find rethink_ee_description)/urdf/electric_gripper/fingers/${r_finger}.xacro" />
+    <xacro:finger_xacro gripper_side="${gripper_side}" finger_side="r" reflect="-1"
+      finger_tip="${r_finger_tip}" finger_grasp="${r_finger_grasp}" />
     <xacro:if value="${finger_length > tip_finger_length}">
-        <xacro:property name="tip_finger_length" value="${finger_length}" scope="local"/>
+      <xacro:property name="tip_finger_length" value="${finger_length}" scope="local" />
     </xacro:if>
     <!-- Electric Gripper Base Joint -->
     <joint name="${side}_gripper_base_fixed" type="fixed">
-      <origin rpy="0 0 0" xyz="0 0 0.025"/>
-      <parent link="${side}_hand"/>
-      <child link="${side}_gripper_base"/>
+      <origin rpy="0 0 0" xyz="0 0 0.025" />
+      <parent link="${side}_hand" />
+      <child link="${side}_gripper_base" />
     </joint>
     <!-- Electric Gripper Tip joint -->
     <joint name="${side}_endpoint" type="fixed">
-      <origin rpy="0 0 0" xyz="0 0 ${tip_finger_length+0.02}"/>
-      <parent link="${side}_gripper_base"/>
-      <child link="${side}_gripper"/>
+      <origin rpy="0 0 0" xyz="0 0 ${tip_finger_length+0.02}" />
+      <parent link="${side}_gripper_base" />
+      <child link="${side}_gripper" />
     </joint>
     <!-- Electric Gripper Tip link -->
     <link name="${side}_gripper">
       <inertial>
-        <origin rpy="0 0 0" xyz="0 0 0"/>
-        <mass value="0.0001"/>
-        <inertia ixx="0" ixy="0" ixz="0" iyy="0" iyz="0" izz="0.0"/>
+        <origin rpy="0 0 0" xyz="0 0 0" />
+        <mass value="0.0001" />
+        <inertia ixx="0" ixy="0" ixz="0" iyy="0" iyz="0" izz="0.0" />
       </inertial>
     </link>
     <!-- Left finger -->
-    <xacro:property name="l_finger_offset" value="${((l_finger_slot-1)*0.0095) -0.011}" scope="local"/>
+    <xacro:property name="l_finger_offset" value="${((l_finger_slot-1)*0.0095) -0.011}"
+      scope="local" />
     <joint name="${gripper_side}_gripper_l_finger_joint" type="prismatic">
-      <origin rpy="0 0 0" xyz="0.0 ${l_finger_offset} 0.02"/>
-      <axis xyz="0 1 0"/>
-      <parent link="${side}_gripper_base"/>
-      <child link="${gripper_side}_gripper_l_finger"/>
-      <limit effort="20.0" lower="0.0" upper="0.020833" velocity="5.0"/>
-      <dynamics damping="0.7" friction="0.0"/>
+      <origin rpy="0 0 0" xyz="0.0 ${l_finger_offset} 0.02" />
+      <axis xyz="0 1 0" />
+      <parent link="${side}_gripper_base" />
+      <child link="${gripper_side}_gripper_l_finger" />
+      <limit effort="20.0" lower="0.0" upper="0.020833" velocity="5.0" />
+      <dynamics damping="0.7" friction="0.0" />
     </joint>
     <!-- Right finger -->
-    <xacro:property name="r_finger_offset" value="${((r_finger_slot-1)*-0.0095) +0.011}" scope="local"/>
+    <xacro:property name="r_finger_offset" value="${((r_finger_slot-1)*-0.0095) +0.011}"
+      scope="local" />
     <joint name="${gripper_side}_gripper_r_finger_joint" type="prismatic">
-      <origin rpy="0 0 0" xyz="0.0 ${r_finger_offset} 0.02"/>
-      <axis xyz="0 1 0"/>
-      <parent link="${side}_gripper_base"/>
-      <child link="${gripper_side}_gripper_r_finger"/>
-      <limit effort="20.0" lower="-0.020833" upper="0.0" velocity="5.0"/>
-      <mimic joint="${gripper_side}_gripper_l_finger_joint" multiplier="-1.0"/>
-      <dynamics damping="0.7" friction="0.0"/>
+      <origin rpy="0 0 0" xyz="0.0 ${r_finger_offset} 0.02" />
+      <axis xyz="0 1 0" />
+      <parent link="${side}_gripper_base" />
+      <child link="${gripper_side}_gripper_r_finger" />
+      <limit effort="20.0" lower="-0.020833" upper="0.0" velocity="5.0" />
+      <mimic joint="${gripper_side}_gripper_l_finger_joint" multiplier="-1.0" />
+      <dynamics damping="0.7" friction="0.0" />
     </joint>
     <transmission name="gripper_${side}1">

File: src/rethink_ee_description/urdf/pneumatic_gripper/pneumatic_gripper_base.xacro (robot description, xacro)
@@ -8,5 +8,5 @@
         <origin rpy="0 ${pi} ${pi}" xyz="0 0 0"/>
         <geometry>
-          <mesh filename="file://$(find rethink_ee_description)/meshes/pneumatic_gripper/pneumatic_gripper_base.DAE"/>
+          <mesh filename="$(find rethink_ee_description)/meshes/pneumatic_gripper/pneumatic_gripper_base.DAE"/>
         </geometry>
       </visual>

File: src/rethink_ee_description/urdf/pneumatic_gripper/rethink_pneumatic_gripper.xacro (robot description, xacro)
@@ -8,5 +8,5 @@
         <origin rpy="0 ${pi} ${pi}" xyz="0 0 0"/>
         <geometry>
-          <mesh filename="file://$(find rethink_ee_description)/meshes/pneumatic_gripper/pneumatic_gripper_w_cup.DAE"/>
+          <mesh filename="$(find rethink_ee_description)/meshes/pneumatic_gripper/pneumatic_gripper_w_cup.DAE"/>
         </geometry>
       </visual>

Commit message: tf runs only once

File: src/baxter_description/urdf/left_end_effector.urdf.xacro (robot description, xacro)
@@ -1,14 +1,13 @@
-<?xml version="1.0"?>
+<?xml version="1.0" ?>
 <robot name="left_end_effector" xmlns:xacro="http://www.ros.org/wiki/xacro">
-  <xacro:include
-    filename="$(find rethink_ee_description)/urdf/electric_gripper/rethink_electric_gripper.xacro" />
+  <xacro:include filename="$(find rethink_ee_description)/urdf/electric_gripper/rethink_electric_gripper.xacro" />
   <xacro:rethink_electric_gripper side="left"
-    l_finger="extended_narrow"
-    l_finger_slot="2"
-    l_finger_tip="paddle_tip"
-    l_finger_grasp="inner"
-    r_finger="extended_narrow"
-    r_finger_slot="2"
-    r_finger_tip="paddle_tip"
-    r_finger_grasp="inner" />
+                                  l_finger="extended_narrow"
+                                  l_finger_slot="2"
+                                  l_finger_tip="paddle_tip"
+                                  l_finger_grasp="inner"
+                                  r_finger="extended_narrow"
+                                  r_finger_slot="2"
+                                  r_finger_tip="paddle_tip"
+                                  r_finger_grasp="inner"/>
 </robot>

File: src/baxter_description/urdf/pedestal/pedestal.xacro (robot description, xacro)
@@ -30,8 +30,9 @@
     <child link="pedestal"/>
   </joint>
-  <xacro:if value="$(arg gazebo)">
-    <!-- When using the pedistal, fix Baxter to Gazebo world with 'base' frame -->
+  <xacro:if value="True">
+    <!-- When using the pedistal, fix Baxter to Webots world with 'base' frame -->
     <link name="world"/>
     <joint name="fixed" type="fixed">
+      <origin rpy="0 0 0" xyz="0.0 0.0 0.927"/>
       <parent link="world"/>
       <child link="base"/>

File: src/baxter_description/urdf/right_end_effector.urdf.xacro (robot description, xacro)
@@ -1,14 +1,13 @@
-<?xml version="1.0"?>
+<?xml version="1.0" ?>
 <robot name="right_end_effector" xmlns:xacro="http://www.ros.org/wiki/xacro">
-  <xacro:include
-    filename="$(find rethink_ee_description)/urdf/electric_gripper/rethink_electric_gripper.xacro" />
+  <xacro:include filename="$(find rethink_ee_description)/urdf/electric_gripper/rethink_electric_gripper.xacro" />
   <xacro:rethink_electric_gripper side="right"
-    l_finger="extended_narrow"
-    l_finger_slot="2"
-    l_finger_tip="paddle_tip"
-    l_finger_grasp="inner"
-    r_finger="extended_narrow"
-    r_finger_slot="2"
-    r_finger_tip="paddle_tip"
-    r_finger_grasp="inner" />
+                                  l_finger="extended_narrow"
+                                  l_finger_slot="2"
+                                  l_finger_tip="paddle_tip"
+                                  l_finger_grasp="inner"
+                                  r_finger="extended_narrow"
+                                  r_finger_slot="2"
+                                  r_finger_tip="paddle_tip"
+                                  r_finger_grasp="inner"/>
 </robot>
