Commit message: both arm joint trajectory working

File: src/baxter_description/urdf/baxter_base/baxter_base.webots.xacro (robot description, xacro)
@@ -2,101 +2,99 @@
 <robot xmlns:xacro="http://www.ros.org/wiki/xacro">
   <xacro:macro name="ros2_control"
-    params="name prefix initial_positions">
-    <ros2_control name="${name}" type="system">
-      <hardware>
-        <plugin>webots_ros2_control::Ros2ControlSystem</plugin>
-      </hardware>
-      <joint name="${prefix}_s0">
-        <command_interface name="position">
-        </command_interface>
-        <state_interface name="position" />
-        <state_interface name="velocity" />
-        <state_interface name="effort" />
-        <param name="initial_position">${initial_positions[prefix + '_s0']}</param>  <!-- initial
+    params="prefix initial_positions">
+    <hardware>
+      <plugin>webots_ros2_control::Ros2ControlSystem</plugin>
+    </hardware>
+    <joint name="${prefix}_s0">
+      <command_interface name="position">
+      </command_interface>
+      <state_interface name="position" />
+      <state_interface name="velocity" />
+      <state_interface name="effort" />
+      <param name="initial_position">${initial_positions[prefix + '_s0']}</param>  <!-- initial
         position
         for the FakeSystem -->
-      </joint>
-      <joint name="${prefix}_s1">
-        <command_interface name="position">
-        </command_interface>
-        <state_interface name="position" />
-        <state_interface name="velocity" />
-        <state_interface name="effort" />
-        <param name="initial_position">${initial_positions[prefix + '_s1']}</param>  <!-- initial
+    </joint>
+    <joint name="${prefix}_s1">
+      <command_interface name="position">
+      </command_interface>
+      <state_interface name="position" />
+      <state_interface name="velocity" />
+      <state_interface name="effort" />
+      <param name="initial_position">${initial_positions[prefix + '_s1']}</param>  <!-- initial
         position
         for the FakeSystem -->
-      </joint>
-      <joint name="${prefix}_e0">
-        <command_interface name="position">
-        </command_interface>
-        <state_interface name="position" />
-        <state_interface name="velocity" />
-        <state_interface name="effort" />
-        <param name="initial_position">${initial_positions[prefix + '_e0']}</param>  <!-- initial
+    </joint>
+    <joint name="${prefix}_e0">
+      <command_interface name="position">
+      </command_interface>
+      <state_interface name="position" />
+      <state_interface name="velocity" />
+      <state_interface name="effort" />
+      <param name="initial_position">${initial_positions[prefix + '_e0']}</param>  <!-- initial
         position
         for the FakeSystem -->
-      </joint>
-      <joint name="${prefix}_e1">
-        <command_interface name="position">
-        </command_interface>
-        <state_interface name="position" />
-        <state_interface name="velocity" />
-        <state_interface name="effort" />
-        <param name="initial_position">${initial_positions[prefix + '_e1']}</param>  <!-- initial
+    </joint>
+    <joint name="${prefix}_e1">
+      <command_interface name="position">
+      </command_interface>
+      <state_interface name="position" />
+      <state_interface name="velocity" />
+      <state_interface name="effort" />
+      <param name="initial_position">${initial_positions[prefix + '_e1']}</param>  <!-- initial
         position
         for the FakeSystem -->
-      </joint>
-      <joint name="${prefix}_w0">
-        <command_interface name="position">
-        </command_interface>
-        <state_interface name="position" />
-        <state_interface name="velocity" />
-        <state_interface name="effort" />
-        <param name="initial_position">${initial_positions[prefix + '_w0']}</param>  <!-- initial
+    </joint>
+    <joint name="${prefix}_w0">
+      <command_interface name="position">
+      </command_interface>
+      <state_interface name="position" />
+      <state_interface name="velocity" />
+      <state_interface name="effort" />
+      <param name="initial_position">${initial_positions[prefix + '_w0']}</param>  <!-- initial
         position
         for the FakeSystem -->
-      </joint>
-      <joint name="${prefix}_w1">
-        <command_interface name="position">
-        </command_interface>
-        <state_interface name="position" />
-        <state_interface name="velocity" />
-        <state_interface name="effort" />
-        <param name="initial_position">${initial_positions[prefix + '_w1']}</param>  <!-- initial
+    </joint>
+    <joint name="${prefix}_w1">
+      <command_interface name="position">
+      </command_interface>
+      <state_interface name="position" />
+      <state_interface name="velocity" />
+      <state_interface name="effort" />
+      <param name="initial_position">${initial_positions[prefix + '_w1']}</param>  <!-- initial
         position
         for the FakeSystem -->
-      </joint>
-      <joint name="${prefix}_w2">
-        <command_interface name="position">
-        </command_interface>
-        <state_interface name="position" />
-        <state_interface name="velocity" />
-        <state_interface name="effort" />
-        <param name="initial_position">${initial_positions[prefix + '_w2']}</param>  <!-- initial
+    </joint>
+    <joint name="${prefix}_w2">
+      <command_interface name="position">
+      </command_interface>
+      <state_interface name="position" />
+      <state_interface name="velocity" />
+      <state_interface name="effort" />
+      <param name="initial_position">${initial_positions[prefix + '_w2']}</param>  <!-- initial
         position
         for the FakeSystem -->
+    </joint>
+    <!-- Baxter Electric EE -->
+    <xacro:if value="${prefix == 'right'}">
+      <joint name="r_gripper_l_finger_joint">
+        <state_interface name="position" />
+        <command_interface name="position" />
       </joint>
-      <!-- Baxter Electric EE -->
-      <xacro:if value="${prefix == 'right'}">
-        <joint name="r_gripper_l_finger_joint">
-          <state_interface name="position" />
-          <command_interface name="position" />
-        </joint>
-        <joint name="r_gripper_r_finger_joint">
-          <state_interface name="position" />
-          <command_interface name="position" />
-        </joint>
-      </xacro:if>
-      <xacro:if value="${prefix == 'left'}">
-        <joint name="r_gripper_l_finger_joint">
-          <state_interface name="position" />
-          <command_interface name="position" />
-        </joint>
-        <joint name="r_gripper_r_finger_joint">
-          <state_interface name="position" />
-          <command_interface name="position" />
-        </joint>
-      </xacro:if>
-    </ros2_control>
+      <joint name="r_gripper_r_finger_joint">
+        <state_interface name="position" />
+        <command_interface name="position" />
+      </joint>
+    </xacro:if>
+    <xacro:if value="${prefix == 'left'}">
+      <joint name="l_gripper_l_finger_joint">
+        <state_interface name="position" />
+        <command_interface name="position" />
+      </joint>
+      <joint name="l_gripper_r_finger_joint">
+        <state_interface name="position" />
+        <command_interface name="position" />
+      </joint>
+    </xacro:if>
   </xacro:macro>
 </robot>

File: src/webots_baxter/resource/urdf/baxter_webots.xacro (robot description, xacro)
@@ -5,10 +5,13 @@
         <plugin type="webots_ros2_control::Ros2Control" />
     </webots>
-    <xacro:property name="initial_positions_file" value="$(find webots_baxter)/config/initial_positions.yaml" />
+    <xacro:property name="initial_positions_file"
+        value="$(find webots_baxter)/config/initial_positions.yaml" />
     <xacro:property name="initial_positions" value="${xacro.load_yaml(initial_positions_file)}" />
     <!-- Baxter Ros2 Control -->
     <xacro:include filename="$(find baxter_description)/urdf/baxter_base/baxter_base.webots.xacro" />
-    <xacro:ros2_control name='WebotsControl' prefix='right' initial_positions="${initial_positions}" />
-    <!-- <xacro:ros2_control name='WebotsControl' prefix='left' initial_positions="${initial_positions}" /> -->
+    <ros2_control name="WebotsControl" type="system">
+        <xacro:ros2_control prefix='right' initial_positions="${initial_positions}" />
+        <xacro:ros2_control prefix='left' initial_positions="${initial_positions}" />
+    </ros2_control>
     <!-- baxter robot -->
     <xacro:include filename="$(find baxter_description)/urdf/baxter.urdf.xacro" />

Commit message: update

File: src/baxter_description/urdf/baxter_base/baxter_base.webots.xacro (robot description, xacro)
@@ -76,4 +76,17 @@
         for the FakeSystem -->
     </joint>
+<!-- Adding Control for HeadPan -->
+    <xacro:if value="${prefix == 'right'}">
+      <joint name="head_pan">
+        <command_interface name="position">
+        </command_interface>
+        <state_interface name="position" />
+        <state_interface name="velocity" />
+        <state_interface name="effort" />
+        <param name="initial_position">${initial_positions['head_pan']}</param>  <!-- initial
+        position
+        for the FakeSystem -->
+      </joint>
+    </xacro:if>
     <!-- Baxter Electric EE -->
     <xacro:if value="${prefix == 'right'}">

File: src/rethink_ee_description/urdf/electric_gripper/fingers/basic_hard_tip.xacro (robot description, xacro)
@@ -10,5 +10,5 @@
         <origin rpy="0 0 ${pi*(g_reflect+1)/2}" xyz="0 0 0"/>
         <geometry>
-          <mesh filename="$(find rethink_ee_description)/meshes/electric_gripper/fingers/basic_hard_tip.DAE" />
+          <mesh filename="package://rethink_ee_description/meshes/electric_gripper/fingers/basic_hard_tip.DAE" />
         </geometry>
       </visual>

File: src/rethink_ee_description/urdf/electric_gripper/fingers/basic_soft_tip.xacro (robot description, xacro)
@@ -10,5 +10,5 @@
         <origin rpy="0 0 ${pi*(g_reflect+1)/2}" xyz="0 0 0"/>
         <geometry>
-          <mesh filename="$(find rethink_ee_description)/meshes/electric_gripper/fingers/basic_soft_tip.DAE" />
+          <mesh filename="package://rethink_ee_description/meshes/electric_gripper/fingers/basic_soft_tip.DAE" />
         </geometry>
       </visual>

File: src/rethink_ee_description/urdf/electric_gripper/fingers/extended_narrow.xacro (robot description, xacro)
@@ -8,5 +8,5 @@
         <origin rpy="0 0 ${-pi/2*(reflect+1)}" xyz="0 0 0"/>
         <geometry>
-          <mesh filename="$(find rethink_ee_description)/meshes/electric_gripper/fingers/extended_narrow.DAE" />
+          <mesh filename="package://rethink_ee_description/meshes/electric_gripper/fingers/extended_narrow.DAE" />
         </geometry>
       </visual>

File: src/rethink_ee_description/urdf/electric_gripper/fingers/extended_wide.xacro (robot description, xacro)
@@ -8,5 +8,5 @@
         <origin rpy="0 0 ${-pi/2*(reflect+1)}" xyz="0 0 0"/>
         <geometry>
-          <mesh filename="$(find rethink_ee_description)/meshes/electric_gripper/fingers/extended_wide.DAE" />
+          <mesh filename="package://rethink_ee_description/meshes/electric_gripper/fingers/extended_wide.DAE" />
         </geometry>
       </visual>

File: src/rethink_ee_description/urdf/electric_gripper/fingers/half_round_tip.xacro (robot description, xacro)
@@ -10,5 +10,5 @@
         <origin rpy="0 0 ${pi*(g_reflect+1)/2}" xyz="0 0 0"/>
         <geometry>
-          <mesh filename="$(find rethink_ee_description)/meshes/electric_gripper/fingers/half_round_tip.DAE" />
+          <mesh filename="package://rethink_ee_description/meshes/electric_gripper/fingers/half_round_tip.DAE" />
         </geometry>
       </visual>

File: src/rethink_ee_description/urdf/electric_gripper/fingers/paddle_tip.xacro (robot description, xacro)
@@ -10,5 +10,5 @@
         <origin rpy="0 0 ${pi*(g_reflect+1)/2}" xyz="0 0 0"/>
         <geometry>
-          <mesh filename="$(find rethink_ee_description)/meshes/electric_gripper/fingers/paddle_tip.DAE" />
+          <mesh filename="package://rethink_ee_description/meshes/electric_gripper/fingers/paddle_tip.DAE" />
         </geometry>
       </visual>

File: src/rethink_ee_description/urdf/electric_gripper/fingers/standard_narrow.xacro (robot description, xacro)
@@ -8,5 +8,5 @@
         <origin rpy="0 0 ${-pi/2*(reflect+1)}" xyz="0 0 0"/>
         <geometry>
-          <mesh filename="$(find rethink_ee_description)/meshes/electric_gripper/fingers/standard_narrow.DAE" />
+          <mesh filename="package://rethink_ee_description/meshes/electric_gripper/fingers/standard_narrow.DAE" />
         </geometry>
       </visual>

File: src/rethink_ee_description/urdf/electric_gripper/fingers/standard_wide.xacro (robot description, xacro)
@@ -8,5 +8,5 @@
         <origin rpy="0 0 ${-pi/2*(reflect+1)}" xyz="0 0 0"/>
         <geometry>
-          <mesh filename="$(find rethink_ee_description)/meshes/electric_gripper/fingers/standard_wide.DAE" />
+          <mesh filename="package://rethink_ee_description/meshes/electric_gripper/fingers/standard_wide.DAE" />
         </geometry>
       </visual>

File: src/rethink_ee_description/urdf/electric_gripper/rethink_electric_gripper.xacro (robot description, xacro)
@@ -10,5 +10,5 @@
         <geometry>
           <mesh
-            filename="$(find rethink_ee_description)/meshes/electric_gripper/electric_gripper_base.DAE" />
+            filename="package://rethink_ee_description/meshes/electric_gripper/electric_gripper_base.DAE" />
         </geometry>
       </visual>

File: src/rethink_ee_description/urdf/pneumatic_gripper/pneumatic_gripper_base.xacro (robot description, xacro)
@@ -8,5 +8,5 @@
         <origin rpy="0 ${pi} ${pi}" xyz="0 0 0"/>
         <geometry>
-          <mesh filename="$(find rethink_ee_description)/meshes/pneumatic_gripper/pneumatic_gripper_base.DAE"/>
+          <mesh filename="package://rethink_ee_description/meshes/pneumatic_gripper/pneumatic_gripper_base.DAE"/>
         </geometry>
       </visual>

File: src/rethink_ee_description/urdf/pneumatic_gripper/rethink_pneumatic_gripper.xacro (robot description, xacro)
@@ -8,5 +8,5 @@
         <origin rpy="0 ${pi} ${pi}" xyz="0 0 0"/>
         <geometry>
-          <mesh filename="$(find rethink_ee_description)/meshes/pneumatic_gripper/pneumatic_gripper_w_cup.DAE"/>
+          <mesh filename="package://rethink_ee_description/meshes/pneumatic_gripper/pneumatic_gripper_w_cup.DAE"/>
         </geometry>
       </visual>
