Commit message: working moveit

File: src/baxter_description/urdf/baxter_base/baxter_base.urdf.xacro (robot description, xacro)
@@ -525,5 +525,5 @@
     <parent link="right_upper_shoulder"/>
     <child link="right_lower_shoulder"/>
-    <limit effort="50.0" lower="-2.147" upper="1.047" velocity="1.5"/>
+    <limit effort="500.0" lower="-2.147" upper="1.047" velocity="1.5"/>
     <dynamics damping="0.7" friction="0.0"/>
   </joint>
@@ -893,5 +893,5 @@
     <parent link="left_upper_shoulder"/>
     <child link="left_lower_shoulder"/>
-    <limit effort="50.0" lower="-2.147" upper="1.047" velocity="1.5"/>
+    <limit effort="100.0" lower="-2.147" upper="1.047" velocity="1.5"/>
     <dynamics damping="0.7" friction="0.0"/>
   </joint>

File: src/webots_baxter/config/srdf/baxter_base.srdf.xacro (robot description, xacro)
@@ -1,8 +1,9 @@
-<?xml version="1.0" encoding="UTF-8"?>
+<?xml version="1.0" ?>
 <!--This does not replace URDF, and is not an extension of URDF.
     This is a format for representing semantic information about the robot structure.
     A URDF file must exist for this robot as well, where the joints and the links that are referenced are defined
 -->
-<robot name="baxter">
+<robot xmlns:xacro="http://www.ros.org/wiki/xacro" name="baxter">
+  <xacro:macro name="baxter_base" params="left_tip_name right_tip_name">
     <!--GROUPS: Representation of a set of joints and links. This can be useful for specifying DOF to plan for, defining arms, end effectors, etc-->
     <!--LINKS: When a link is specified, the parent joint of that link (if it exists) is automatically included-->
@@ -10,25 +11,11 @@
     <!--CHAINS: When a chain is specified, all the links along the chain (including endpoints) are included in the group. Additionally, all the joints that are parents to included links are also included. This means that joints along the chain and the parent joint of the base link are included in the group-->
     <!--SUBGROUPS: Groups can also be formed by referencing to already defined group names-->
+    <xacro:arg name="left_tip_name" default="left_gripper"/>
+    <xacro:arg name="right_tip_name" default="right_gripper"/>
     <group name="left_arm">
-        <chain base_link="torso" tip_link="left_gripper" />
-        <!-- <link name="left_gripper"/>
-        <joint name="left_s0"/>
-        <joint name="left_s1"/>
-        <joint name="left_e0"/>
-        <joint name="left_e1"/>
-        <joint name="left_w0"/>
-        <joint name="left_w1"/>
-        <joint name="left_w2"/> -->
+        <chain base_link="torso" tip_link="$(arg left_tip_name)" />
     </group>
     <group name="right_arm">
-        <chain base_link="torso" tip_link="right_gripper" />
-        <!-- <link name="right_gripper"/>
-        <joint name="right_s0"/>
-        <joint name="right_s1"/>
-        <joint name="right_e0"/>
-        <joint name="right_e1"/>
-        <joint name="right_w0"/>
-        <joint name="right_w1"/>
-        <joint name="right_w2"/> -->
+        <chain base_link="torso" tip_link="$(arg right_tip_name)" />
     </group>
     <group name="both_arms">
@@ -36,41 +23,37 @@
         <group name="left_arm" />
     </group>
-    <!-- <group name="left_ee">
-        <chain base_link="left_hand" tip_link="left_gripper" />
-        <joint name="l_gripper_l_finger_joint"/>
-        <joint name="l_gripper_r_finger_joint"/>
-    </group>
-    <group name="right_ee">
-        <chain base_link="left_hand" tip_link="right_gripper" />
-        <joint name="r_gripper_l_finger_joint"/>
-        <joint name="r_gripper_r_finger_joint"/>
-    </group> -->
-    <group name="head">
-        <joint name="head_pan"/>
-    </group>
+    <group name="left_hand">
+        <chain base_link="left_hand" tip_link="$(arg left_tip_name)" />
+    </group>
+    <group name="right_hand">
+        <chain base_link="right_hand" tip_link="$(arg right_tip_name)" />
+    </group>
+    <!--END EFFECTOR: Purpose: Represent information about an end effector.-->
+    <end_effector name="left_hand_eef" parent_link="$(arg left_tip_name)" group="left_hand" parent_group="left_arm" />
+    <end_effector name="right_hand_eef" parent_link="$(arg right_tip_name)" group="right_hand" parent_group="right_arm" />
     <!--GROUP STATES: Purpose: Define a named state for a particular group, in terms of joint values. This is useful to define states like 'folded arms'-->
-    <group_state name="left_arm_home" group="left_arm">
-        <joint name="left_e0" value="0"/>
-        <joint name="left_e1" value="0"/>
-        <joint name="left_s0" value="0"/>
-        <joint name="left_s1" value="0"/>
-        <joint name="left_w0" value="0"/>
-        <joint name="left_w1" value="0"/>
-        <joint name="left_w2" value="0"/>
+    <group_state name="left_neutral" group="left_arm">
+        <joint name="left_e0" value="0" />
+        <joint name="left_e1" value="0.75" />
+        <joint name="left_s0" value="0" />
+        <joint name="left_s1" value="-0.55" />
+        <joint name="left_w0" value="0" />
+        <joint name="left_w1" value="1.26" />
+        <joint name="left_w2" value="0" />
     </group_state>
-    <group_state name="right_arm_home" group="right_arm">
-        <joint name="right_e0" value="0"/>
-        <joint name="right_e1" value="0"/>
-        <joint name="right_s0" value="0"/>
-        <joint name="right_s1" value="0"/>
-        <joint name="right_w0" value="0"/>
-        <joint name="right_w1" value="0"/>
-        <joint name="right_w2" value="0"/>
+    <group_state name="right_neutral" group="right_arm">
+        <joint name="right_e0" value="0" />
+        <joint name="right_e1" value="0.75" />
+        <joint name="right_s0" value="0" />
+        <joint name="right_s1" value="-0.55" />
+        <joint name="right_w0" value="0" />
+        <joint name="right_w1" value="1.26" />
+        <joint name="right_w2" value="0" />
     </group_state>
     <!--END EFFECTOR: Purpose: Represent information about an end effector.-->
-    <!-- <end_effector name="left_gripper" parent_link="left_gripper" group="left_ee" parent_group="left_arm"/>
-    <end_effector name="right_gripper" parent_link="right_gripper" group="right_ee" parent_group="right_arm"/> -->
-    <!--VIRTUAL JOINT: Purpose: this element defines a virtual joint between a robot link and an external frame of reference (considered fixed with respect to the robot)-->
-    <virtual_joint name="virtual_joint" type="fixed" parent_frame="virtual_world" child_link="base"/>
+     <!--VIRTUAL JOINT: Purpose: this element defines a virtual joint between a robot link and an external frame of reference (considered fixed with respect to the robot)-->
+    <virtual_joint name="world_joint" type="floating" parent_frame="world" child_link="base" />
+    <!--PASSIVE JOINT: Purpose: this element is used to mark joints that are not actuated-->
+    <passive_joint name="world_joint" />
     <!--DISABLE COLLISIONS: By default it is assumed that any link of the robot could potentially come into collision with any other link in the robot. This tag disables collision checking between a specified pair of links. -->
     <disable_collisions link1="collision_head_link_1" link2="collision_head_link_2" reason="Adjacent" />
@@ -305,112 +288,4 @@
     <disable_collisions link1="sonar_ring" link2="torso" reason="Adjacent" />
     <disable_collisions link1="screen" link2="display" reason="Adjacent" />
-    <disable_collisions link1="l_gripper_l_finger" link2="l_gripper_l_finger_tip" reason="Adjacent"/>
-    <disable_collisions link1="l_gripper_l_finger" link2="l_gripper_r_finger" reason="Default"/>
-    <disable_collisions link1="l_gripper_l_finger" link2="l_gripper_r_finger_tip" reason="Never"/>
-    <disable_collisions link1="l_gripper_l_finger" link2="left_gripper_base" reason="Adjacent"/>
-    <disable_collisions link1="l_gripper_l_finger" link2="left_hand" reason="Never"/>
-    <disable_collisions link1="l_gripper_l_finger" link2="left_lower_elbow" reason="Never"/>
-    <disable_collisions link1="l_gripper_l_finger" link2="left_lower_forearm" reason="Never"/>
-    <disable_collisions link1="l_gripper_l_finger" link2="left_upper_elbow_visual" reason="Never"/>
-    <disable_collisions link1="l_gripper_l_finger" link2="left_upper_forearm" reason="Never"/>
-    <disable_collisions link1="l_gripper_l_finger" link2="left_upper_forearm_visual" reason="Never"/>
-    <disable_collisions link1="l_gripper_l_finger" link2="left_wrist" reason="Never"/>
-    <disable_collisions link1="l_gripper_l_finger" link2="r_gripper_l_finger_tip" reason="Never"/>
-    <disable_collisions link1="l_gripper_l_finger" link2="screen" reason="Never"/>
-    <disable_collisions link1="l_gripper_l_finger_tip" link2="l_gripper_r_finger" reason="Never"/>
-    <disable_collisions link1="l_gripper_l_finger_tip" link2="l_gripper_r_finger_tip" reason="Never"/>
-    <disable_collisions link1="l_gripper_l_finger_tip" link2="left_gripper_base" reason="Never"/>
-    <disable_collisions link1="l_gripper_l_finger_tip" link2="left_hand" reason="Never"/>
-    <disable_collisions link1="l_gripper_l_finger_tip" link2="left_lower_elbow" reason="Never"/>
-    <disable_collisions link1="l_gripper_l_finger_tip" link2="left_lower_forearm" reason="Never"/>
-    <disable_collisions link1="l_gripper_l_finger_tip" link2="left_upper_elbow_visual" reason="Never"/>
-    <disable_collisions link1="l_gripper_l_finger_tip" link2="left_upper_forearm" reason="Never"/>
-    <disable_collisions link1="l_gripper_l_finger_tip" link2="left_upper_forearm_visual" reason="Never"/>
-    <disable_collisions link1="l_gripper_l_finger_tip" link2="left_wrist" reason="Never"/>
-    <disable_collisions link1="l_gripper_l_finger_tip" link2="r_gripper_l_finger_tip" reason="Never"/>
-    <disable_collisions link1="l_gripper_l_finger_tip" link2="screen" reason="Never"/>
-    <disable_collisions link1="l_gripper_l_finger_tip" link2="sonar_ring" reason="Never"/>
-    <disable_collisions link1="l_gripper_r_finger" link2="l_gripper_r_finger_tip" reason="Adjacent"/>
-    <disable_collisions link1="l_gripper_r_finger" link2="left_gripper_base" reason="Adjacent"/>
-    <disable_collisions link1="l_gripper_r_finger" link2="left_hand" reason="Never"/>
-    <disable_collisions link1="l_gripper_r_finger" link2="left_lower_elbow" reason="Never"/>
-    <disable_collisions link1="l_gripper_r_finger" link2="left_lower_forearm" reason="Never"/>
-    <disable_collisions link1="l_gripper_r_finger" link2="left_upper_elbow_visual" reason="Never"/>
-    <disable_collisions link1="l_gripper_r_finger" link2="left_upper_forearm" reason="Never"/>
-    <disable_collisions link1="l_gripper_r_finger" link2="left_upper_forearm_visual" reason="Never"/>
-    <disable_collisions link1="l_gripper_r_finger" link2="left_wrist" reason="Never"/>
-    <disable_collisions link1="l_gripper_r_finger" link2="r_gripper_l_finger_tip" reason="Never"/>
-    <disable_collisions link1="l_gripper_r_finger" link2="screen" reason="Never"/>
-    <disable_collisions link1="l_gripper_r_finger" link2="sonar_ring" reason="Never"/>
-    <disable_collisions link1="l_gripper_r_finger_tip" link2="left_gripper_base" reason="Never"/>
-    <disable_collisions link1="l_gripper_r_finger_tip" link2="left_hand" reason="Never"/>
-    <disable_collisions link1="l_gripper_r_finger_tip" link2="left_lower_elbow" reason="Never"/>
-    <disable_collisions link1="l_gripper_r_finger_tip" link2="left_lower_forearm" reason="Never"/>
-    <disable_collisions link1="l_gripper_r_finger_tip" link2="left_upper_elbow_visual" reason="Never"/>
-    <disable_collisions link1="l_gripper_r_finger_tip" link2="left_upper_forearm" reason="Never"/>
-    <disable_collisions link1="l_gripper_r_finger_tip" link2="left_upper_forearm_visual" reason="Never"/>
-    <disable_collisions link1="l_gripper_r_finger_tip" link2="left_wrist" reason="Never"/>
-    <disable_collisions link1="l_gripper_r_finger_tip" link2="r_gripper_l_finger_tip" reason="Never"/>
-    <disable_collisions link1="l_gripper_r_finger_tip" link2="right_hand" reason="Never"/>
-    <disable_collisions link1="l_gripper_r_finger_tip" link2="screen" reason="Never"/>
-    <disable_collisions link1="l_gripper_r_finger_tip" link2="sonar_ring" reason="Never"/>
-    <disable_collisions link1="left_gripper_base" link2="left_hand" reason="Adjacent"/>
-    <disable_collisions link1="left_gripper_base" link2="left_lower_elbow" reason="Never"/>
-    <disable_collisions link1="left_gripper_base" link2="left_lower_forearm" reason="Never"/>
-    <disable_collisions link1="left_gripper_base" link2="left_upper_elbow_visual" reason="Never"/>
-    <disable_collisions link1="left_gripper_base" link2="left_upper_forearm" reason="Never"/>
-    <disable_collisions link1="left_gripper_base" link2="left_upper_forearm_visual" reason="Never"/>
-    <disable_collisions link1="left_gripper_base" link2="left_wrist" reason="Never"/>
-    <disable_collisions link1="r_gripper_l_finger" link2="r_gripper_l_finger_tip" reason="Adjacent"/>
-    <disable_collisions link1="r_gripper_l_finger" link2="r_gripper_r_finger" reason="Default"/>
-    <disable_collisions link1="r_gripper_l_finger" link2="r_gripper_r_finger_tip" reason="Never"/>
-    <disable_collisions link1="r_gripper_l_finger" link2="right_gripper_base" reason="Adjacent"/>
-    <disable_collisions link1="r_gripper_l_finger" link2="right_hand" reason="Never"/>
-    <disable_collisions link1="r_gripper_l_finger" link2="right_lower_elbow" reason="Never"/>
-    <disable_collisions link1="r_gripper_l_finger" link2="right_lower_forearm" reason="Never"/>
-    <disable_collisions link1="r_gripper_l_finger" link2="right_upper_elbow_visual" reason="Never"/>
-    <disable_collisions link1="r_gripper_l_finger" link2="right_upper_forearm" reason="Never"/>
-    <disable_collisions link1="r_gripper_l_finger" link2="right_upper_forearm_visual" reason="Never"/>
-    <disable_collisions link1="r_gripper_l_finger" link2="right_wrist" reason="Never"/>
-    <disable_collisions link1="r_gripper_l_finger" link2="screen" reason="Never"/>
-    <disable_collisions link1="r_gripper_l_finger" link2="sonar_ring" reason="Never"/>
-    <disable_collisions link1="r_gripper_l_finger_tip" link2="r_gripper_r_finger" reason="Never"/>
-    <disable_collisions link1="r_gripper_l_finger_tip" link2="r_gripper_r_finger_tip" reason="Never"/>
-    <disable_collisions link1="r_gripper_l_finger_tip" link2="right_gripper_base" reason="Never"/>
-    <disable_collisions link1="r_gripper_l_finger_tip" link2="right_hand" reason="Never"/>
-    <disable_collisions link1="r_gripper_l_finger_tip" link2="right_lower_elbow" reason="Never"/>
-    <disable_collisions link1="r_gripper_l_finger_tip" link2="right_lower_forearm" reason="Never"/>
-    <disable_collisions link1="r_gripper_l_finger_tip" link2="right_upper_elbow_visual" reason="Never"/>
-    <disable_collisions link1="r_gripper_l_finger_tip" link2="right_upper_forearm" reason="Never"/>
-    <disable_collisions link1="r_gripper_l_finger_tip" link2="right_upper_forearm_visual" reason="Never"/>
-    <disable_collisions link1="r_gripper_l_finger_tip" link2="right_wrist" reason="Never"/>
-    <disable_collisions link1="r_gripper_l_finger_tip" link2="screen" reason="Never"/>
-    <disable_collisions link1="r_gripper_r_finger" link2="r_gripper_r_finger_tip" reason="Adjacent"/>
-    <disable_collisions link1="r_gripper_r_finger" link2="right_gripper_base" reason="Adjacent"/>
-    <disable_collisions link1="r_gripper_r_finger" link2="right_hand" reason="Never"/>
-    <disable_collisions link1="r_gripper_r_finger" link2="right_lower_elbow" reason="Never"/>
-    <disable_collisions link1="r_gripper_r_finger" link2="right_lower_forearm" reason="Never"/>
-    <disable_collisions link1="r_gripper_r_finger" link2="right_upper_elbow_visual" reason="Never"/>
-    <disable_collisions link1="r_gripper_r_finger" link2="right_upper_forearm" reason="Never"/>
-    <disable_collisions link1="r_gripper_r_finger" link2="right_upper_forearm_visual" reason="Never"/>
-    <disable_collisions link1="r_gripper_r_finger" link2="right_wrist" reason="Never"/>
-    <disable_collisions link1="r_gripper_r_finger" link2="screen" reason="Never"/>
-    <disable_collisions link1="r_gripper_r_finger" link2="sonar_ring" reason="Never"/>
-    <disable_collisions link1="r_gripper_r_finger_tip" link2="right_gripper_base" reason="Never"/>
-    <disable_collisions link1="r_gripper_r_finger_tip" link2="right_hand" reason="Never"/>
-    <disable_collisions link1="r_gripper_r_finger_tip" link2="right_lower_elbow" reason="Never"/>
-    <disable_collisions link1="r_gripper_r_finger_tip" link2="right_lower_forearm" reason="Never"/>
-    <disable_collisions link1="r_gripper_r_finger_tip" link2="right_upper_elbow_visual" reason="Never"/>
-    <disable_collisions link1="r_gripper_r_finger_tip" link2="right_upper_forearm" reason="Never"/>
-    <disable_collisions link1="r_gripper_r_finger_tip" link2="right_upper_forearm_visual" reason="Never"/>
-    <disable_collisions link1="r_gripper_r_finger_tip" link2="right_wrist" reason="Never"/>
-    <disable_collisions link1="r_gripper_r_finger_tip" link2="screen" reason="Never"/>
-    <disable_collisions link1="r_gripper_r_finger_tip" link2="sonar_ring" reason="Never"/>
-    <disable_collisions link1="right_gripper_base" link2="right_hand" reason="Adjacent"/>
-    <disable_collisions link1="right_gripper_base" link2="right_lower_elbow" reason="Never"/>
-    <disable_collisions link1="right_gripper_base" link2="right_lower_forearm" reason="Never"/>
-    <disable_collisions link1="right_gripper_base" link2="right_upper_elbow_visual" reason="Never"/>
-    <disable_collisions link1="right_gripper_base" link2="right_upper_forearm" reason="Never"/>
-    <disable_collisions link1="right_gripper_base" link2="right_upper_forearm_visual" reason="Never"/>
-    <disable_collisions link1="right_gripper_base" link2="right_wrist" reason="Never"/>
+</xacro:macro>
 </robot>

File: src/webots_baxter/resource/urdf/baxter.ros2_control.xacro (robot description, xacro)
@@ -10,6 +10,4 @@
       </command_interface>
       <state_interface name="position" />
-      <state_interface name="velocity" />
-      <state_interface name="effort" />
       <param name="initial_position">${initial_positions[prefix + '_s0']}</param>  <!-- initial
         position
@@ -20,6 +18,4 @@
       </command_interface>
       <state_interface name="position" />
-      <state_interface name="velocity" />
-      <state_interface name="effort" />
       <param name="initial_position">${initial_positions[prefix + '_s1']}</param>  <!-- initial
         position
@@ -30,6 +26,4 @@
       </command_interface>
       <state_interface name="position" />
-      <state_interface name="velocity" />
-      <state_interface name="effort" />
       <param name="initial_position">${initial_positions[prefix + '_e0']}</param>  <!-- initial
         position
@@ -40,6 +34,4 @@
       </command_interface>
       <state_interface name="position" />
-      <state_interface name="velocity" />
-      <state_interface name="effort" />
       <param name="initial_position">${initial_positions[prefix + '_e1']}</param>  <!-- initial
         position
@@ -50,6 +42,4 @@
       </command_interface>
       <state_interface name="position" />
-      <state_interface name="velocity" />
-      <state_interface name="effort" />
       <param name="initial_position">${initial_positions[prefix + '_w0']}</param>  <!-- initial
         position
@@ -60,6 +50,4 @@
       </command_interface>
       <state_interface name="position" />
-      <state_interface name="velocity" />
-      <state_interface name="effort" />
       <param name="initial_position">${initial_positions[prefix + '_w1']}</param>  <!-- initial
         position
@@ -70,6 +58,4 @@
       </command_interface>
       <state_interface name="position" />
-      <state_interface name="velocity" />
-      <state_interface name="effort" />
       <param name="initial_position">${initial_positions[prefix + '_w2']}</param>  <!-- initial
         position
@@ -82,6 +68,4 @@
         </command_interface>
         <state_interface name="position" />
-        <state_interface name="velocity" />
-        <state_interface name="effort" />
         <param name="initial_position">${initial_positions['head_pan']}</param>  <!-- initial
         position
