Commit message: Update

File: src/webots_baxter/resource/urdf/baxter_webots.xacro (robot description, xacro)
@@ -6,5 +6,5 @@
     </webots>
     <xacro:property name="initial_positions_file" value="$(find webots_baxter)/config/initial_positions.yaml" />
-    <xacro:property name="initial_positions" value="${load_yaml(initial_positions_file)}" />
+    <xacro:property name="initial_positions" value="${xacro.load_yaml(initial_positions_file)}" />
     <!-- Baxter Ros2 Control -->
     <xacro:include filename="$(find baxter_description)/urdf/baxter_base/baxter_base.webots.xacro" />

Commit message: update

File: src/webots_baxter/resource/urdf/baxter_webots.xacro (robot description, xacro)
@@ -7,7 +7,7 @@
     <xacro:property name="initial_positions_file"
         value="$(find webots_baxter)/config/initial_positions.yaml" />
-    <xacro:property name="initial_positions" value="${xacro.load_yaml(initial_positions_file)}" />
+    <xacro:property name="initial_positions" value="${xacro.load_yaml(initial_positions_file)['initial_positions']}" />
     <!-- Baxter Ros2 Control -->
-    <xacro:include filename="$(find baxter_description)/urdf/baxter_base/baxter_base.webots.xacro" />
+    <xacro:include filename="$(find webots_baxter)/resource/urdf/baxter.ros2_control.xacro" />
     <ros2_control name="WebotsControl" type="system">
         <xacro:ros2_control prefix='right' initial_positions="${initial_positions}" />
