Commit message: All components loading into webots and rviz

File: src/webots_baxter/resource/baxter/urdf/baxter_webots.xacro (robot description, xacro)
@@ -9,5 +9,5 @@
     <xacro:property name="initial_positions" value="${xacro.load_yaml(initial_positions_file)['initial_positions']}" />
     <!-- Baxter Ros2 Control -->
-    <xacro:include filename="$(find webots_baxter)/resource/urdf/baxter.ros2_control.xacro" />
+    <xacro:include filename="$(find webots_baxter)/resource/baxter/urdf/baxter.ros2_control.xacro" />
     <ros2_control name="WebotsControl" type="system">
         <xacro:ros2_control prefix='right' initial_positions="${initial_positions}" />

File: src/webots_baxter/resource/kinect/urdf/kinect.urdf (robot description, URDF)
Before this commit: robot Vision, 4 links, 3 joints
Links:
- link solid: geometry collision mesh filename=package://webots_baxter/resource/kinect/meshes/kinect.dae; visual mesh filename=package://webots_baxter/resource/kinect/meshes/kinect.dae

File: src/webots_baxter/resource/lego/1x1.urdf.xacro (robot description, xacro)
@@ -7,5 +7,4 @@
             <box size="0.032 0.032 0.021"/>
            </geometry>
-           <material name="blue" />
         </visual>
         <collision>

Commit message: Kinect and table to spawn with robot

File: src/webots_baxter/resource/baxter/urdf/baxter_webots.xacro (robot description, xacro)
@@ -2,10 +2,16 @@
 <robot name="baxter" xmlns:xacro="http://wiki.ros.org/xacro">
     <!-- Custom Baxter Xacro-->
+    <!-- math constants -->
+    <xacro:property name="M_PI" value="3.1415926535897931" />
+    <!-- Parameters -->
+    <xacro:property name="initial_positions_file"
+        value="$(find webots_baxter)/config/initial_positions.yaml" />
+    <xacro:property name="initial_positions"
+        value="${xacro.load_yaml(initial_positions_file)['initial_positions']}" />
+    <!-- Baxter and Kinect Plugin -->
     <webots>
         <plugin type="webots_ros2_control::Ros2Control" />
+        <xacro:include filename="$(find webots_baxter)/resource/kinect/urdf/kinect_control.urdf" />
     </webots>
-    <xacro:property name="initial_positions_file"
-        value="$(find webots_baxter)/config/initial_positions.yaml" />
-    <xacro:property name="initial_positions" value="${xacro.load_yaml(initial_positions_file)['initial_positions']}" />
     <!-- Baxter Ros2 Control -->
     <xacro:include filename="$(find webots_baxter)/resource/baxter/urdf/baxter.ros2_control.xacro" />
@@ -16,3 +22,8 @@
     <!-- baxter robot -->
     <xacro:include filename="$(find baxter_description)/urdf/baxter.urdf.xacro" />
+    <!-- Kinect Links -->
+    <xacro:include filename="$(find webots_baxter)/resource/kinect/urdf/kinect.urdf.xacro" />
+    <xacro:kinect xyz="0.8 0 1.5" rpy="0 ${M_PI/2} ${M_PI}" parent_frame="world" />
+    <!-- Table  -->
+    <xacro:include filename="$(find webots_baxter)/resource/table/urdf/table.urdf.xacro" />
 </robot>

File: src/webots_baxter/resource/kinect/urdf/kinect.urdf.xacro (robot description, xacro)
@@ -1,9 +1,133 @@
 <?xml version="1.0"?>
-<robot name="Kinect" xmlns:xacro="http://wiki.ros.org/xacro">
-    <!-- Webots Plugin -->
-    <xacro:include filename="$(find webots_baxter)/resource/kinect/urdf/kinect_control.urdf" />
-    <!-- Kinect Links -->
-    <xacro:include filename="$(find webots_baxter)/resource/kinect/urdf/kinect.urdf" />
-    <!-- Table Links -->
-    <xacro:include filename="$(find webots_baxter)/resource/table/urdf/table.urdf.xacro" />
+<robot name="Kinect" xmlns:xi="http://www.w3.org/2001/XInclude"
+    xmlns:gazebo="http://playerstage.sourceforge.net/gazebo/xmlschema/#gz"
+    xmlns:model="http://playerstage.sourceforge.net/gazebo/xmlschema/#model"
+    xmlns:sensor="http://playerstage.sourceforge.net/gazebo/xmlschema/#sensor"
+    xmlns:body="http://playerstage.sourceforge.net/gazebo/xmlschema/#body"
+    xmlns:geom="http://playerstage.sourceforge.net/gazebo/xmlschema/#geom"
+    xmlns:joint="http://playerstage.sourceforge.net/gazebo/xmlschema/#joint"
+    xmlns:controller="http://playerstage.sourceforge.net/gazebo/xmlschema/#controller"
+    xmlns:interface="http://playerstage.sourceforge.net/gazebo/xmlschema/#interface"
+    xmlns:rendering="http://playerstage.sourceforge.net/gazebo/xmlschema/#rendering"
+    xmlns:renderable="http://playerstage.sourceforge.net/gazebo/xmlschema/#renderable"
+    xmlns:physics="http://playerstage.sourceforge.net/gazebo/xmlschema/#physics"
+    xmlns:xacro="http://ros.org/wiki/xacro">
+  <!-- math constants -->
+  <xacro:property name="M_PI" value="3.1415926535897931" />
+  <xacro:macro name="kinect" params="xyz rpy parent_frame" >
+  <joint name="base_camera_joint" type="fixed">
+    <origin xyz="${xyz}" rpy="${rpy}" />
+    <parent link="${parent_frame}" />
+    <origin xyz="0 0 0" rpy="0 0 0" />
+    <child link="camera_link" />
+  </joint>
+  <link name="camera_link">
+    <inertial>
+      <mass value="0.01" />
+      <origin xyz="0 0 0" />
+      <inertia ixx="0.001" ixy="0.0" ixz="0.0"
+        iyy="0.001" iyz="0.0"
+        izz="0.001" />
+    </inertial>
+    <visual>
+      <origin xyz=" 0 0 0 " rpy="0 0 0" />
+      <geometry>
+        <mesh filename="package://webots_baxter/resource/kinect/meshes/kinect.dae"/>
+      </geometry>
+    </visual>
+    <collision>
+      <origin xyz="0.0 0.0 0.0" rpy="0 0 0" />
+      <geometry>
+        <box size="0.0730 .2760 0.0720"/>
+      </geometry>
+    </collision>
+  </link>
+  <joint name="camera_depth_joint" type="fixed">
+    <origin xyz="0 0.011 0" rpy="0 0 0" />
+    <parent link="camera_link" />
+    <child link="camera_depth_frame" />
+  </joint>
+  <link name="camera_depth_frame">
+    <inertial>
+      <mass value="0.01" />
+      <origin xyz="0 0 0" />
+      <inertia ixx="0.001" ixy="0.0" ixz="0.0"
+        iyy="0.001" iyz="0.0"
+        izz="0.001" />
+    </inertial>
+  </link>
+  <joint name="camera_depth_optical_joint" type="fixed">
+    <origin xyz="0 0 0" rpy="${-M_PI/2} 0 ${-M_PI/2}" />
+    <parent link="camera_depth_frame" />
+    <child link="camera_depth_optical_frame" />
+  </joint>
+  <link name="camera_depth_optical_frame">
+    <inertial>
+      <mass value="0.001" />
+      <origin xyz="0 0 0" />
+      <inertia ixx="0.0001" ixy="0.0" ixz="0.0"
+        iyy="0.0001" iyz="0.0"
+        izz="0.0001" />
+    </inertial>
+  </link>
+  <joint name="camera_rgb_joint" type="fixed">
+    <origin xyz="0 -0.012 0" rpy="0 0 0" />
+    <parent link="camera_link" />
+    <child link="camera_rgb_frame" />
+  </joint>
+  <link name="camera_rgb_frame">
+    <inertial>
+      <mass value="0.001" />
+      <origin xyz="0 0 0" />
+      <inertia ixx="0.0001" ixy="0.0" ixz="0.0"
+        iyy="0.0001" iyz="0.0"
+        izz="0.0001" />
+    </inertial>
+  </link>
+  <joint name="camera_rgb_optical_joint" type="fixed">
+    <origin xyz="0 0 0" rpy="${-M_PI/2} 0 ${-M_PI/2}" />
+    <parent link="camera_rgb_frame" />
+    <child link="camera_rgb_optical_frame" />
+  </joint>
+  <link name="camera_rgb_optical_frame">
+    <inertial>
+      <mass value="0.001" />
+      <origin xyz="0 0 0" />
+      <inertia ixx="0.0001" ixy="0.0" ixz="0.0"
+        iyy="0.0001" iyz="0.0"
+        izz="0.0001" />
+    </inertial>
+  </link>
+  <!-- Camera Sensor -->
+    <!-- reference is the link camera is attached to  -->
+    <gazebo reference="camera_rgb_optical_frame">
+        <sensor name="camera_rgb_frame" type="camera">
+            <camera>
+                <horizontal_fov>1</horizontal_fov>
+                <image>
+                    <format>R8G8B8</format>
+                    <width>640</width>
+                    <height>480</height>
+                </image>
+            </camera>
+        </sensor>
+    </gazebo>
+    <!-- Depth Sensor -->
+    <gazebo reference="camera_depth_optical_frame">
+        <sensor name="camera_depth_frame" type="depth">
+            <camera>
+                <horizontal_fov>1</horizontal_fov>
+                <image>
+                    <format>R8G8B8</format>
+                    <width>640</width>
+                    <height>480</height>
+                </image>
+                <clip>
+                    <near>0.05</near>
+                    <far>3</far>
+                  </clip>
+            </camera>
+        </sensor>
+    </gazebo>
+</xacro:macro>
 </robot>

Commit message: adding 2nd kinect

File: src/webots_baxter/resource/baxter/urdf/baxter_webots.xacro (robot description, xacro)
@@ -12,5 +12,6 @@
     <webots>
         <plugin type="webots_ros2_control::Ros2Control" />
-        <xacro:include filename="$(find webots_baxter)/resource/kinect/urdf/kinect_control.urdf" />
+        <!-- <xacro:include filename="$(find webots_baxter)/resource/kinect/urdf/kinect_control.urdf" /> -->
+        <xacro:include filename="$(find webots_baxter)/resource/kinect_1/urdf/kinect_control.urdf" />
     </webots>
     <!-- Baxter Ros2 Control -->
@@ -23,7 +24,19 @@
     <xacro:include filename="$(find baxter_description)/urdf/baxter.urdf.xacro" />
     <!-- Kinect Links -->
-    <xacro:include filename="$(find webots_baxter)/resource/kinect/urdf/kinect.urdf.xacro" />
-    <xacro:kinect xyz="0.8 0 1.5" rpy="0 ${M_PI/2} ${M_PI}" parent_frame="world" />
+    <!-- <xacro:include filename="$(find webots_baxter)/resource/kinect/urdf/kinect.urdf.xacro" />
+    <xacro:kinect xyz="0.8 0 1.5" rpy="0 ${M_PI/2} ${M_PI}" parent_frame="world" /> -->
     <!-- Table  -->
     <xacro:include filename="$(find webots_baxter)/resource/table/urdf/table.urdf.xacro" />
+    <!-- Source Table and Kinect -->
+    <!-- Kinect Links -->
+    <link name="world_1"/>
+    <joint name="world_1_fixed" type="fixed">
+      <origin rpy="0 0 0" xyz="0.0 3.0 0.0"/>
+      <parent link="world"/>
+      <child link="world_1"/>
+    </joint>
+    <xacro:include filename="$(find webots_baxter)/resource/kinect_1/urdf/kinect.urdf.xacro" />
+    <xacro:kinect xyz="0.8 0 1.5" rpy="0 ${M_PI/2} ${M_PI}" parent_frame="world_1" />
+    <!-- Table  -->
+    <xacro:include filename="$(find webots_baxter)/resource/table_1/urdf/table.urdf.xacro" />
 </robot>

Commit message: adding 2nd kinect

File: src/webots_baxter/resource/baxter/urdf/baxter_webots.xacro (robot description, xacro)
@@ -12,5 +12,5 @@
     <webots>
         <plugin type="webots_ros2_control::Ros2Control" />
-        <!-- <xacro:include filename="$(find webots_baxter)/resource/kinect/urdf/kinect_control.urdf" /> -->
+        <xacro:include filename="$(find webots_baxter)/resource/kinect/urdf/kinect_control.urdf" />
         <xacro:include filename="$(find webots_baxter)/resource/kinect_1/urdf/kinect_control.urdf" />
     </webots>
@@ -24,6 +24,6 @@
     <xacro:include filename="$(find baxter_description)/urdf/baxter.urdf.xacro" />
     <!-- Kinect Links -->
-    <!-- <xacro:include filename="$(find webots_baxter)/resource/kinect/urdf/kinect.urdf.xacro" />
-    <xacro:kinect xyz="0.8 0 1.5" rpy="0 ${M_PI/2} ${M_PI}" parent_frame="world" /> -->
+    <xacro:include filename="$(find webots_baxter)/resource/kinect/urdf/kinect.urdf.xacro" />
+    <xacro:kinect xyz="0.8 0 1.5" rpy="0 ${M_PI/2} ${M_PI}" parent_frame="world" />
     <!-- Table  -->
     <xacro:include filename="$(find webots_baxter)/resource/table/urdf/table.urdf.xacro" />
@@ -37,5 +37,5 @@
     </joint>
     <xacro:include filename="$(find webots_baxter)/resource/kinect_1/urdf/kinect.urdf.xacro" />
-    <xacro:kinect xyz="0.8 0 1.5" rpy="0 ${M_PI/2} ${M_PI}" parent_frame="world_1" />
+    <xacro:kinect_1 xyz="0.8 0 1.5" rpy="0 ${M_PI/2} ${M_PI}" parent_frame="world_1" />
     <!-- Table  -->
     <xacro:include filename="$(find webots_baxter)/resource/table_1/urdf/table.urdf.xacro" />

File: src/webots_baxter/resource/kinect_1/urdf/kinect.urdf.xacro (robot description, xacro)
@@ -15,12 +15,12 @@
   <!-- math constants -->
   <xacro:property name="M_PI" value="3.1415926535897931" />
-  <xacro:macro name="kinect" params="xyz rpy parent_frame" >
-  <joint name="base_camera_joint" type="fixed">
+  <xacro:macro name="kinect_1" params="xyz rpy parent_frame" >
+  <joint name="base_camera_joint_1" type="fixed">
     <origin xyz="${xyz}" rpy="${rpy}" />
     <parent link="${parent_frame}" />
     <origin xyz="0 0 0" rpy="0 0 0" />
-    <child link="camera_link" />
+    <child link="camera_link_1" />
   </joint>
-  <link name="camera_link">
+  <link name="camera_link_1">
     <inertial>
       <mass value="0.01" />
@@ -43,10 +43,10 @@
     </collision>
   </link>
-  <joint name="camera_depth_joint" type="fixed">
+  <joint name="camera_depth_joint_1" type="fixed">
     <origin xyz="0 0.011 0" rpy="0 0 0" />
-    <parent link="camera_link" />
-    <child link="camera_depth_frame" />
+    <parent link="camera_link_1" />
+    <child link="camera_depth_frame_1" />
   </joint>
-  <link name="camera_depth_frame">
+  <link name="camera_depth_frame_1">
     <inertial>
       <mass value="0.01" />
@@ -57,10 +57,10 @@
     </inertial>
   </link>
-  <joint name="camera_depth_optical_joint" type="fixed">
+  <joint name="camera_depth_optical_joint_1" type="fixed">
     <origin xyz="0 0 0" rpy="${-M_PI/2} 0 ${-M_PI/2}" />
-    <parent link="camera_depth_frame" />
-    <child link="camera_depth_optical_frame" />
+    <parent link="camera_depth_frame_1" />
+    <child link="camera_depth_optical_frame_1" />
   </joint>
-  <link name="camera_depth_optical_frame">
+  <link name="camera_depth_optical_frame_1">
     <inertial>
       <mass value="0.001" />
@@ -71,10 +71,10 @@
     </inertial>
   </link>
-  <joint name="camera_rgb_joint" type="fixed">
+  <joint name="camera_rgb_joint_1" type="fixed">
     <origin xyz="0 -0.012 0" rpy="0 0 0" />
-    <parent link="camera_link" />
-    <child link="camera_rgb_frame" />
+    <parent link="camera_link_1" />
+    <child link="camera_rgb_frame_1" />
   </joint>
-  <link name="camera_rgb_frame">
+  <link name="camera_rgb_frame_1">
     <inertial>
       <mass value="0.001" />
@@ -85,10 +85,10 @@
     </inertial>
   </link>
-  <joint name="camera_rgb_optical_joint" type="fixed">
+  <joint name="camera_rgb_optical_joint_1" type="fixed">
     <origin xyz="0 0 0" rpy="${-M_PI/2} 0 ${-M_PI/2}" />
-    <parent link="camera_rgb_frame" />
-    <child link="camera_rgb_optical_frame" />
+    <parent link="camera_rgb_frame_1" />
+    <child link="camera_rgb_optical_frame_1" />
   </joint>
-  <link name="camera_rgb_optical_frame">
+  <link name="camera_rgb_optical_frame_1">
     <inertial>
       <mass value="0.001" />
@@ -101,6 +101,6 @@
   <!-- Camera Sensor -->
     <!-- reference is the link camera is attached to  -->
-    <gazebo reference="camera_rgb_optical_frame">
-        <sensor name="camera_rgb_frame" type="camera">
+    <gazebo reference="camera_rgb_optical_frame_1">
+        <sensor name="camera_rgb_frame_1" type="camera">
             <camera>
                 <horizontal_fov>1</horizontal_fov>
@@ -114,6 +114,6 @@
     </gazebo>
     <!-- Depth Sensor -->
-    <gazebo reference="camera_depth_optical_frame">
-        <sensor name="camera_depth_frame" type="depth">
+    <gazebo reference="camera_depth_optical_frame_1">
+        <sensor name="camera_depth_frame_1" type="depth">
             <camera>
                 <horizontal_fov>1</horizontal_fov>
