Commit message: working complete cycle

File: src/webots_baxter/config/srdf/baxter_base.srdf.xacro (robot description, xacro)
@@ -259,4 +259,5 @@
         <disable_collisions link1="pedestal" link2="screen" reason="Never" />
         <disable_collisions link1="pedestal" link2="sonar_ring" reason="Never" />
+        <disable_collisions link1="pedestal" link2="desk" reason="Never" />
         <disable_collisions link1="pedestal" link2="torso" reason="Adjacent" />
         <disable_collisions link1="right_hand" link2="right_hand_accelerometer" reason="Never" />

File: src/webots_baxter/resource/table/urdf/table.urdf.xacro (robot description, xacro)
@@ -66,5 +66,5 @@
     <parent link="world" />
     <child link="desk" />
-    <origin xyz="0.8 0 0" rpy="0 0 0" />
+    <origin xyz="0.5 0 0" rpy="0 0 0" />
   </joint>
 </robot>

File: src/webots_baxter/resource/table_1/urdf/table.urdf.xacro (robot description, xacro)
@@ -66,5 +66,5 @@
     <parent link="world_1" />
     <child link="desk_1" />
-    <origin xyz="0.8 0 0" rpy="0 0 0" />
+    <origin xyz="0.5 0 0" rpy="0 0 0" />
   </joint>
 </robot>
