Commit message: Working Gripper Control

File: src/rethink_ee_description/urdf/electric_gripper/rethink_electric_gripper.xacro (robot description, xacro)
@@ -83,5 +83,5 @@
       <child link="${gripper_side}_gripper_r_finger" />
       <limit effort="20.0" lower="-0.020833" upper="0.0" velocity="5.0" />
-      <mimic joint="${gripper_side}_gripper_l_finger_joint" multiplier="-1.0" />
+      <!-- <mimic joint="${gripper_side}_gripper_l_finger_joint" multiplier="-1.0" /> -->
       <dynamics damping="0.7" friction="0.0" />
     </joint>
