Commit message: Working Gripper Control

File: src/webots_baxter/config/srdf/baxter_base.srdf.xacro (robot description, xacro)
@@ -1,291 +1,353 @@
-<?xml version="1.0" ?>
+<?xml version="1.0"?>
 <!--This does not replace URDF, and is not an extension of URDF.
     This is a format for representing semantic information about the robot structure.
-    A URDF file must exist for this robot as well, where the joints and the links that are referenced are defined
+    A URDF file must exist for this robot as well, where the joints and the links that are referenced
+are defined
 -->
 <robot xmlns:xacro="http://www.ros.org/wiki/xacro" name="baxter">
-  <xacro:macro name="baxter_base" params="left_tip_name right_tip_name">
-    <!--GROUPS: Representation of a set of joints and links. This can be useful for specifying DOF to plan for, defining arms, end effectors, etc-->
-    <!--LINKS: When a link is specified, the parent joint of that link (if it exists) is automatically included-->
-    <!--JOINTS: When a joint is specified, the child link of that joint (which will always exist) is automatically included-->
-    <!--CHAINS: When a chain is specified, all the links along the chain (including endpoints) are included in the group. Additionally, all the joints that are parents to included links are also included. This means that joints along the chain and the parent joint of the base link are included in the group-->
-    <!--SUBGROUPS: Groups can also be formed by referencing to already defined group names-->
-    <xacro:arg name="left_tip_name" default="left_gripper"/>
-    <xacro:arg name="right_tip_name" default="right_gripper"/>
-    <group name="left_arm">
-        <chain base_link="torso" tip_link="$(arg left_tip_name)" />
-    </group>
-    <group name="right_arm">
-        <chain base_link="torso" tip_link="$(arg right_tip_name)" />
-    </group>
-    <group name="both_arms">
-        <group name="right_arm" />
-        <group name="left_arm" />
-    </group>
-    <group name="left_hand">
-        <chain base_link="left_hand" tip_link="$(arg left_tip_name)" />
-    </group>
-    <group name="right_hand">
-        <chain base_link="right_hand" tip_link="$(arg right_tip_name)" />
-    </group>
-    <!--END EFFECTOR: Purpose: Represent information about an end effector.-->
-    <end_effector name="left_hand_eef" parent_link="$(arg left_tip_name)" group="left_hand" parent_group="left_arm" />
-    <end_effector name="right_hand_eef" parent_link="$(arg right_tip_name)" group="right_hand" parent_group="right_arm" />
-    <!--GROUP STATES: Purpose: Define a named state for a particular group, in terms of joint values. This is useful to define states like 'folded arms'-->
-    <group_state name="left_neutral" group="left_arm">
-        <joint name="left_e0" value="0" />
-        <joint name="left_e1" value="0.75" />
-        <joint name="left_s0" value="0" />
-        <joint name="left_s1" value="-0.55" />
-        <joint name="left_w0" value="0" />
-        <joint name="left_w1" value="1.26" />
-        <joint name="left_w2" value="0" />
-    </group_state>
-    <group_state name="right_neutral" group="right_arm">
-        <joint name="right_e0" value="0" />
-        <joint name="right_e1" value="0.75" />
-        <joint name="right_s0" value="0" />
-        <joint name="right_s1" value="-0.55" />
-        <joint name="right_w0" value="0" />
-        <joint name="right_w1" value="1.26" />
-        <joint name="right_w2" value="0" />
-    </group_state>
-    <!--END EFFECTOR: Purpose: Represent information about an end effector.-->
-     <!--VIRTUAL JOINT: Purpose: this element defines a virtual joint between a robot link and an external frame of reference (considered fixed with respect to the robot)-->
-    <virtual_joint name="world_joint" type="floating" parent_frame="world" child_link="base" />
-    <!--PASSIVE JOINT: Purpose: this element is used to mark joints that are not actuated-->
-    <passive_joint name="world_joint" />
-    <!--DISABLE COLLISIONS: By default it is assumed that any link of the robot could potentially come into collision with any other link in the robot. This tag disables collision checking between a specified pair of links. -->
-    <disable_collisions link1="collision_head_link_1" link2="collision_head_link_2" reason="Adjacent" />
-    <disable_collisions link1="collision_head_link_1" link2="head" reason="Never" />
-    <disable_collisions link1="collision_head_link_1" link2="left_lower_shoulder" reason="Never" />
-    <disable_collisions link1="collision_head_link_1" link2="left_upper_elbow" reason="Never" />
-    <disable_collisions link1="collision_head_link_1" link2="left_upper_shoulder" reason="Never" />
-    <disable_collisions link1="collision_head_link_1" link2="pedestal" reason="Never" />
-    <disable_collisions link1="collision_head_link_1" link2="right_upper_elbow_visual" reason="Never" />
-    <disable_collisions link1="collision_head_link_1" link2="right_lower_shoulder" reason="Never" />
-    <disable_collisions link1="collision_head_link_1" link2="right_upper_shoulder" reason="Never" />
-    <disable_collisions link1="collision_head_link_1" link2="screen" reason="Never" />
-    <disable_collisions link1="collision_head_link_1" link2="sonar_ring" reason="Never" />
-    <disable_collisions link1="collision_head_link_1" link2="torso" reason="Adjacent" />
-    <disable_collisions link1="collision_head_link_1" link2="display" reason="Adjacent" />
-    <disable_collisions link1="collision_head_link_2" link2="head" reason="Never" />
-    <disable_collisions link1="collision_head_link_2" link2="left_upper_shoulder" reason="Never" />
-    <disable_collisions link1="collision_head_link_2" link2="pedestal" reason="Never" />
-    <disable_collisions link1="collision_head_link_2" link2="right_lower_shoulder" reason="Never" />
-    <disable_collisions link1="collision_head_link_2" link2="right_upper_elbow" reason="Never" />
-    <disable_collisions link1="collision_head_link_2" link2="right_upper_shoulder" reason="Never" />
-    <disable_collisions link1="collision_head_link_2" link2="screen" reason="Never" />
-    <disable_collisions link1="collision_head_link_2" link2="sonar_ring" reason="Never" />
-    <disable_collisions link1="collision_head_link_2" link2="torso" reason="Adjacent" />
-    <disable_collisions link1="collision_head_link_2" link2="display" reason="Adjacent" />
-    <disable_collisions link1="head" link2="left_hand_camera" reason="Never" />
-    <disable_collisions link1="head" link2="left_hand_range" reason="Never" />
-    <disable_collisions link1="head" link2="left_lower_shoulder" reason="Never" />
-    <disable_collisions link1="head" link2="left_upper_elbow" reason="Never" />
-    <disable_collisions link1="head" link2="left_upper_elbow_visual" reason="Never" />
-    <disable_collisions link1="head" link2="left_upper_shoulder" reason="Never" />
-    <disable_collisions link1="head" link2="pedestal" reason="Never" />
-    <disable_collisions link1="head" link2="right_hand_camera" reason="Never" />
-    <disable_collisions link1="head" link2="right_hand_range" reason="Never" />
-    <disable_collisions link1="head" link2="right_lower_shoulder" reason="Never" />
-    <disable_collisions link1="head" link2="right_upper_elbow" reason="Never" />
-    <disable_collisions link1="head" link2="right_upper_elbow_visual" reason="Never" />
-    <disable_collisions link1="head" link2="right_upper_shoulder" reason="Never" />
-    <disable_collisions link1="head" link2="screen" reason="Adjacent" />
-    <disable_collisions link1="head" link2="sonar_ring" reason="Never" />
-    <disable_collisions link1="head" link2="torso" reason="Adjacent" />
-    <disable_collisions link1="left_hand" link2="left_hand_camera" reason="Adjacent" />
-    <disable_collisions link1="left_hand" link2="left_hand_range" reason="Adjacent" />
-    <disable_collisions link1="left_hand" link2="left_lower_elbow" reason="Never" />
-    <disable_collisions link1="left_hand" link2="left_lower_forearm" reason="Never" />
-    <disable_collisions link1="left_hand" link2="left_upper_elbow_visual" reason="Never" />
-    <disable_collisions link1="left_hand" link2="left_upper_forearm" reason="Never" />
-    <disable_collisions link1="left_hand" link2="left_upper_forearm_visual" reason="Never" />
-    <disable_collisions link1="left_hand" link2="left_wrist" reason="Adjacent" />
-    <disable_collisions link1="left_hand" link2="pedestal" reason="Never" />
-    <disable_collisions link1="left_hand" link2="left_hand_accelerometer" reason="Never" />
-    <disable_collisions link1="left_hand_camera" link2="left_hand_range" reason="Never" />
-    <disable_collisions link1="left_hand_camera" link2="left_lower_elbow" reason="Never" />
-    <disable_collisions link1="left_hand_camera" link2="left_lower_forearm" reason="Never" />
-    <disable_collisions link1="left_hand_camera" link2="left_upper_elbow" reason="Never" />
-    <disable_collisions link1="left_hand_camera" link2="left_upper_elbow_visual" reason="Never" />
-    <disable_collisions link1="left_hand_camera" link2="left_upper_forearm" reason="Never" />
-    <disable_collisions link1="left_hand_camera" link2="left_upper_forearm_visual" reason="Never" />
-    <disable_collisions link1="left_hand_camera" link2="left_wrist" reason="Never" />
-    <disable_collisions link1="left_hand_camera" link2="right_hand_camera" reason="Never" />
-    <disable_collisions link1="left_hand_camera" link2="right_hand_range" reason="Never" />
-    <disable_collisions link1="left_hand_camera" link2="right_lower_forearm" reason="Never" />
-    <disable_collisions link1="left_hand_camera" link2="screen" reason="Never" />
-    <disable_collisions link1="left_hand_camera" link2="sonar_ring" reason="Never" />
-    <disable_collisions link1="left_hand_range" link2="left_lower_elbow" reason="Never" />
-    <disable_collisions link1="left_hand_range" link2="left_lower_forearm" reason="Never" />
-    <disable_collisions link1="left_hand_range" link2="left_upper_elbow_visual" reason="Never" />
-    <disable_collisions link1="left_hand_range" link2="left_upper_forearm" reason="Never" />
-    <disable_collisions link1="left_wrist" link2="left_hand_accelerometer" reason="Never" />
-    <disable_collisions link1="left_wrist" link2="left_hand" reason="Never" />
-    <disable_collisions link1="left_wrist" link2="left_upper_forearm" reason="Never" />
-    <disable_collisions link1="left_wrist" link2="left_upper_forearm_visual" reason="Never" />
-    <disable_collisions link1="left_wrist" link2="pedestal" reason="Never" />
-    <disable_collisions link1="left_wrist" link2="pedestal" reason="Never" />
-    <disable_collisions link1="left_hand_range" link2="left_upper_forearm_visual" reason="Never" />
-    <disable_collisions link1="left_hand_range" link2="left_wrist" reason="Never" />
-    <disable_collisions link1="left_hand_range" link2="right_hand_camera" reason="Never" />
-    <disable_collisions link1="left_hand_range" link2="right_hand_range" reason="Never" />
-    <disable_collisions link1="left_hand_range" link2="screen" reason="Never" />
-    <disable_collisions link1="left_hand_range" link2="sonar_ring" reason="Never" />
-    <disable_collisions link1="left_lower_elbow" link2="left_lower_forearm" reason="Never" />
-    <disable_collisions link1="left_lower_elbow" link2="left_lower_shoulder" reason="Never" />
-    <disable_collisions link1="left_lower_elbow" link2="left_upper_elbow" reason="Adjacent" />
-    <disable_collisions link1="left_lower_elbow" link2="left_upper_elbow_visual" reason="Never" />
-    <disable_collisions link1="left_lower_elbow" link2="left_upper_forearm" reason="Adjacent" />
-    <disable_collisions link1="left_lower_elbow" link2="left_upper_forearm_visual" reason="Adjacent" />
-    <disable_collisions link1="left_lower_elbow" link2="left_wrist" reason="Never" />
-    <disable_collisions link1="left_lower_elbow" link2="right_lower_shoulder" reason="Never" />
-    <disable_collisions link1="left_lower_elbow" link2="right_upper_shoulder" reason="Never" />
-    <disable_collisions link1="left_lower_forearm" link2="left_lower_shoulder" reason="Never" />
-    <disable_collisions link1="left_lower_forearm" link2="left_upper_elbow_visual" reason="Never" />
-    <disable_collisions link1="left_lower_forearm" link2="left_upper_forearm" reason="Adjacent" />
-    <disable_collisions link1="left_lower_forearm" link2="left_upper_forearm_visual" reason="Never" />
-    <disable_collisions link1="left_lower_forearm" link2="left_wrist" reason="Adjacent" />
-    <disable_collisions link1="left_lower_forearm" link2="sonar_ring" reason="Never" />
-    <disable_collisions link1="left_lower_forearm" link2="pedestal" reason="Never" />
-    <disable_collisions link1="left_lower_shoulder" link2="torso" reason="Never" />
-    <disable_collisions link1="left_lower_shoulder" link2="left_upper_elbow" reason="Adjacent" />
-    <disable_collisions link1="left_lower_shoulder" link2="left_upper_elbow_visual" reason="Adjacent" />
-    <disable_collisions link1="left_lower_shoulder" link2="left_upper_forearm" reason="Never" />
-    <disable_collisions link1="left_lower_shoulder" link2="left_upper_shoulder" reason="Adjacent" />
-    <disable_collisions link1="left_lower_shoulder" link2="pedestal" reason="Never" />
-    <disable_collisions link1="left_lower_shoulder" link2="right_lower_shoulder" reason="Never" />
-    <disable_collisions link1="left_lower_shoulder" link2="right_upper_elbow" reason="Never" />
-    <disable_collisions link1="left_lower_shoulder" link2="right_upper_shoulder" reason="Never" />
-    <disable_collisions link1="left_lower_shoulder" link2="screen" reason="Never" />
-    <disable_collisions link1="left_lower_shoulder" link2="sonar_ring" reason="Never" />
-    <disable_collisions link1="left_upper_elbow" link2="left_upper_elbow_visual" reason="Never" />
-    <disable_collisions link1="left_upper_elbow" link2="pedestal" reason="Never" />
-    <disable_collisions link1="left_upper_elbow" link2="left_upper_shoulder" reason="Never" />
-    <disable_collisions link1="left_upper_elbow" link2="right_lower_shoulder" reason="Never" />
-    <disable_collisions link1="left_upper_elbow" link2="right_upper_elbow" reason="Never" />
-    <disable_collisions link1="left_upper_elbow" link2="right_upper_shoulder" reason="Never" />
-    <disable_collisions link1="left_upper_elbow" link2="screen" reason="Never" />
-    <disable_collisions link1="left_upper_elbow" link2="sonar_ring" reason="Never" />
-    <disable_collisions link1="left_upper_elbow" link2="torso" reason="Never" />
-    <disable_collisions link1="left_upper_elbow_visual" link2="left_upper_forearm_visual" reason="Never" />
-    <disable_collisions link1="left_upper_elbow_visual" link2="left_upper_forearm" reason="Never" />
-    <disable_collisions link1="left_upper_elbow_visual" link2="left_upper_shoulder" reason="Never" />
-    <disable_collisions link1="left_upper_elbow_visual" link2="left_wrist" reason="Never" />
-    <disable_collisions link1="left_upper_elbow_visual" link2="pedestal" reason="Never" />
-    <disable_collisions link1="left_upper_elbow_visual" link2="right_lower_shoulder" reason="Never" />
-    <disable_collisions link1="left_upper_elbow_visual" link2="right_upper_shoulder" reason="Never" />
-    <disable_collisions link1="left_upper_elbow_visual" link2="sonar_ring" reason="Never" />
-    <disable_collisions link1="left_upper_forearm" link2="left_upper_forearm_visual" reason="Default" />
-    <disable_collisions link1="left_upper_forearm" link2="left_wrist" reason="Never" />
-    <disable_collisions link1="left_upper_forearm" link2="pedestal" reason="Never" />
-    <disable_collisions link1="left_upper_forearm_visual" link2="torso" reason="Never" />
-    <disable_collisions link1="left_upper_shoulder" link2="pedestal" reason="Never" />
-    <disable_collisions link1="left_upper_shoulder" link2="right_lower_elbow" reason="Never" />
-    <disable_collisions link1="left_upper_shoulder" link2="right_lower_shoulder" reason="Never" />
-    <disable_collisions link1="left_upper_shoulder" link2="right_upper_elbow" reason="Never" />
-    <disable_collisions link1="left_upper_shoulder" link2="right_upper_elbow_visual" reason="Never" />
-    <disable_collisions link1="left_upper_shoulder" link2="right_upper_shoulder" reason="Never" />
-    <disable_collisions link1="left_upper_shoulder" link2="screen" reason="Never" />
-    <disable_collisions link1="left_upper_shoulder" link2="sonar_ring" reason="Never" />
-    <disable_collisions link1="left_upper_shoulder" link2="torso" reason="Adjacent" />
-    <disable_collisions link1="pedestal" link2="right_hand_accelerometer" reason="Never" />
-    <disable_collisions link1="pedestal" link2="right_hand_camera" reason="Default" />
-    <disable_collisions link1="pedestal" link2="right_hand_range" reason="Default" />
-    <disable_collisions link1="pedestal" link2="right_lower_elbow" reason="Default" />
-    <disable_collisions link1="pedestal" link2="right_lower_shoulder" reason="Never" />
-    <disable_collisions link1="pedestal" link2="right_upper_elbow" reason="Never" />
-    <disable_collisions link1="pedestal" link2="right_upper_forearm" reason="Never" />
-    <disable_collisions link1="pedestal" link2="right_upper_forearm_visual" reason="Default" />
-    <disable_collisions link1="pedestal" link2="right_upper_shoulder" reason="Never" />
-    <disable_collisions link1="pedestal" link2="left_hand_accelerometer" reason="Never" />
-    <disable_collisions link1="pedestal" link2="left_hand_camera" reason="Default" />
-    <disable_collisions link1="pedestal" link2="left_hand_range" reason="Default" />
-    <disable_collisions link1="pedestal" link2="left_lower_elbow" reason="Default" />
-    <disable_collisions link1="pedestal" link2="left_lower_shoulder" reason="Never" />
-    <disable_collisions link1="pedestal" link2="left_upper_elbow" reason="Never" />
-    <disable_collisions link1="pedestal" link2="left_upper_forearm" reason="Never" />
-    <disable_collisions link1="pedestal" link2="left_upper_forearm_visual" reason="Default" />
-    <disable_collisions link1="pedestal" link2="left_upper_shoulder" reason="Never" />
-    <disable_collisions link1="pedestal" link2="screen" reason="Never" />
-    <disable_collisions link1="pedestal" link2="sonar_ring" reason="Never" />
-    <disable_collisions link1="pedestal" link2="torso" reason="Adjacent" />
-    <disable_collisions link1="right_hand" link2="right_hand_accelerometer" reason="Never" />
-    <disable_collisions link1="right_hand" link2="right_hand_camera" reason="Adjacent" />
-    <disable_collisions link1="right_hand" link2="right_hand_range" reason="Adjacent" />
-    <disable_collisions link1="right_hand" link2="right_lower_elbow" reason="Never" />
-    <disable_collisions link1="right_hand" link2="right_lower_forearm" reason="Never" />
-    <disable_collisions link1="right_hand" link2="right_upper_elbow_visual" reason="Never" />
-    <disable_collisions link1="right_hand" link2="right_upper_forearm" reason="Never" />
-    <disable_collisions link1="right_hand" link2="right_upper_forearm_visual" reason="Never" />
-    <disable_collisions link1="right_hand" link2="right_wrist" reason="Adjacent" />
-    <disable_collisions link1="right_hand" link2="pedestal" reason="Never" />
-    <disable_collisions link1="right_hand" link2="right_hand_accelerometer" reason="Never" />
-    <disable_collisions link1="right_hand_camera" link2="right_hand_range" reason="Never" />
-    <disable_collisions link1="right_hand_camera" link2="right_lower_elbow" reason="Never" />
-    <disable_collisions link1="right_hand_camera" link2="right_lower_forearm" reason="Never" />
-    <disable_collisions link1="right_hand_camera" link2="right_upper_elbow_visual" reason="Never" />
-    <disable_collisions link1="right_hand_camera" link2="right_upper_forearm" reason="Never" />
-    <disable_collisions link1="right_hand_camera" link2="right_upper_forearm_visual" reason="Never" />
-    <disable_collisions link1="right_hand_camera" link2="right_wrist" reason="Never" />
-    <disable_collisions link1="right_hand_camera" link2="screen" reason="Never" />
-    <disable_collisions link1="right_hand_camera" link2="sonar_ring" reason="Never" />
-    <disable_collisions link1="right_hand_range" link2="right_lower_elbow" reason="Never" />
-    <disable_collisions link1="right_hand_range" link2="right_lower_forearm" reason="Never" />
-    <disable_collisions link1="right_hand_range" link2="right_upper_elbow" reason="Never" />
-    <disable_collisions link1="right_hand_range" link2="right_upper_elbow_visual" reason="Never" />
-    <disable_collisions link1="right_hand_range" link2="right_upper_forearm" reason="Never" />
-    <disable_collisions link1="right_wrist" link2="right_hand_accelerometer" reason="Never" />
-    <disable_collisions link1="right_wrist" link2="right_upper_forearm" reason="Never" />
-    <disable_collisions link1="right_wrist" link2="right_upper_forearm_visual" reason="Never" />
-    <disable_collisions link1="right_wrist" link2="pedestal" reason="Never" />
-    <disable_collisions link1="right_hand_range" link2="right_upper_forearm_visual" reason="Never" />
-    <disable_collisions link1="right_hand_range" link2="right_wrist" reason="Never" />
-    <disable_collisions link1="right_hand_range" link2="screen" reason="Never" />
-    <disable_collisions link1="right_hand_range" link2="sonar_ring" reason="Never" />
-    <disable_collisions link1="right_lower_elbow" link2="right_lower_forearm" reason="Never" />
-    <disable_collisions link1="right_lower_elbow" link2="right_lower_shoulder" reason="Never" />
-    <disable_collisions link1="right_lower_elbow" link2="right_upper_elbow" reason="Adjacent" />
-    <disable_collisions link1="right_lower_elbow" link2="right_upper_elbow_visual" reason="Never" />
-    <disable_collisions link1="right_lower_elbow" link2="right_upper_forearm" reason="Adjacent" />
-    <disable_collisions link1="right_lower_elbow" link2="right_upper_forearm_visual" reason="Adjacent" />
-    <disable_collisions link1="right_lower_elbow" link2="right_wrist" reason="Never" />
-    <disable_collisions link1="right_lower_elbow" link2="sonar_ring" reason="Never" />
-    <disable_collisions link1="right_lower_forearm" link2="right_lower_shoulder" reason="Never" />
-    <disable_collisions link1="right_lower_forearm" link2="right_upper_elbow_visual" reason="Never" />
-    <disable_collisions link1="right_lower_forearm" link2="right_upper_forearm" reason="Adjacent" />
-    <disable_collisions link1="right_lower_forearm" link2="right_upper_forearm_visual" reason="Never" />
-    <disable_collisions link1="right_lower_forearm" link2="right_wrist" reason="Adjacent" />
-    <disable_collisions link1="right_lower_forearm" link2="pedestal" reason="Never" />
-    <disable_collisions link1="right_lower_shoulder" link2="torso" reason="Never" />
-    <disable_collisions link1="right_lower_shoulder" link2="right_upper_elbow" reason="Adjacent" />
-    <disable_collisions link1="right_lower_shoulder" link2="right_upper_elbow_visual" reason="Adjacent" />
-    <disable_collisions link1="right_lower_shoulder" link2="right_upper_forearm" reason="Never" />
-    <disable_collisions link1="right_lower_shoulder" link2="right_upper_shoulder" reason="Adjacent" />
-    <disable_collisions link1="right_lower_shoulder" link2="screen" reason="Never" />
-    <disable_collisions link1="right_lower_shoulder" link2="sonar_ring" reason="Never" />
-    <disable_collisions link1="right_upper_elbow" link2="right_upper_elbow_visual" reason="Never" />
-    <disable_collisions link1="right_upper_elbow" link2="right_upper_shoulder" reason="Never" />
-    <disable_collisions link1="right_upper_elbow" link2="screen" reason="Never" />
-    <disable_collisions link1="right_upper_elbow" link2="sonar_ring" reason="Never" />
-    <disable_collisions link1="right_upper_elbow" link2="torso" reason="Never" />
-    <disable_collisions link1="right_upper_elbow_visual" link2="right_upper_forearm_visual" reason="Never" />
-    <disable_collisions link1="right_upper_elbow_visual" link2="right_upper_shoulder" reason="Never" />
-    <disable_collisions link1="right_upper_elbow_visual" link2="right_wrist" reason="Never" />
-    <disable_collisions link1="right_upper_elbow_visual" link2="sonar_ring" reason="Never" />
-    <disable_collisions link1="right_upper_elbow_visual" link2="right_upper_forearm" reason="Never" />
-    <disable_collisions link1="right_upper_elbow_visual" link2="pedestal" reason="Never" />
-    <disable_collisions link1="right_upper_forearm" link2="right_upper_forearm_visual" reason="Default" />
-    <disable_collisions link1="right_upper_forearm" link2="right_wrist" reason="Never" />
-    <disable_collisions link1="right_upper_forearm_visual" link2="torso" reason="Never" />
-    <disable_collisions link1="right_upper_shoulder" link2="screen" reason="Never" />
-    <disable_collisions link1="right_upper_shoulder" link2="sonar_ring" reason="Never" />
-    <disable_collisions link1="right_upper_shoulder" link2="torso" reason="Adjacent" />
-    <disable_collisions link1="screen" link2="sonar_ring" reason="Never" />
-    <disable_collisions link1="screen" link2="torso" reason="Never" />
-    <disable_collisions link1="sonar_ring" link2="torso" reason="Adjacent" />
-    <disable_collisions link1="screen" link2="display" reason="Adjacent" />
-</xacro:macro>
+    <xacro:macro name="baxter_base" params="left_tip_name right_tip_name">
+        <!--GROUPS:
+        Representation of a set of joints and links. This can be useful for specifying DOF to plan
+        for, defining arms, end effectors, etc-->
+        <!--LINKS:
+        When a link is specified, the parent joint of that link (if it exists) is automatically
+        included-->
+        <!--JOINTS:
+        When a joint is specified, the child link of that joint (which will always exist) is
+        automatically included-->
+        <!--CHAINS:
+        When a chain is specified, all the links along the chain (including endpoints) are included
+        in the group. Additionally, all the joints that are parents to included links are also
+        included. This means that joints along the chain and the parent joint of the base link are
+        included in the group-->
+        <!--SUBGROUPS:
+        Groups can also be formed by referencing to already defined group names-->
+        <xacro:arg name="left_tip_name" default="left_gripper" />
+        <xacro:arg name="right_tip_name" default="right_gripper" />
+        <group name="left_arm">
+            <chain base_link="torso" tip_link="$(arg left_tip_name)" />
+        </group>
+        <group name="right_arm">
+            <chain base_link="torso" tip_link="$(arg right_tip_name)" />
+        </group>
+        <group name="both_arms">
+            <group name="right_arm" />
+            <group name="left_arm" />
+        </group>
+        <group name="left_hand">
+            <!-- <chain base_link="left_hand" tip_link="$(arg left_tip_name)" /> -->
+            <joint name="l_gripper_l_finger_joint" />
+            <joint name="l_gripper_r_finger_joint" />
+        </group>
+        <group name="right_hand">
+            <!-- <chain base_link="right_hand" tip_link="$(arg right_tip_name)" /> -->
+            <joint name="r_gripper_l_finger_joint" />
+            <joint name="r_gripper_r_finger_joint" />
+        </group>
+        <!--END
+        EFFECTOR: Purpose: Represent information about an end effector.-->
+        <end_effector name="left_hand_eef" parent_link="$(arg left_tip_name)" group="left_hand"
+            parent_group="left_arm" />
+        <end_effector name="right_hand_eef" parent_link="$(arg right_tip_name)" group="right_hand"
+            parent_group="right_arm" />
+        <!--GROUP
+        STATES: Purpose: Define a named state for a particular group, in terms of joint values. This
+        is useful to define states like 'folded arms'-->
+        <group_state name="left_neutral" group="left_arm">
+            <joint name="left_e0" value="0" />
+            <joint name="left_e1" value="0.75" />
+            <joint name="left_s0" value="0" />
+            <joint name="left_s1" value="-0.55" />
+            <joint name="left_w0" value="0" />
+            <joint name="left_w1" value="1.26" />
+            <joint name="left_w2" value="0" />
+        </group_state>
+        <group_state name="right_neutral" group="right_arm">
+            <joint name="right_e0" value="0" />
+            <joint name="right_e1" value="0.75" />
+            <joint name="right_s0" value="0" />
+            <joint name="right_s1" value="-0.55" />
+            <joint name="right_w0" value="0" />
+            <joint name="right_w1" value="1.26" />
+            <joint name="right_w2" value="0" />
+        </group_state>
+        <!--END
+        EFFECTOR: Purpose: Represent information about an end effector.-->
+        <!--VIRTUAL
+        JOINT: Purpose: this element defines a virtual joint between a robot link and an external
+        frame of reference (considered fixed with respect to the robot)-->
+        <virtual_joint name="world_joint" type="floating" parent_frame="world" child_link="base" />
+        <!--PASSIVE
+        JOINT: Purpose: this element is used to mark joints that are not actuated-->
+        <passive_joint name="world_joint" />
+        <!--DISABLE
+        COLLISIONS: By default it is assumed that any link of the robot could potentially come into
+        collision with any other link in the robot. This tag disables collision checking between a
+        specified pair of links. -->
+        <disable_collisions link1="collision_head_link_1" link2="collision_head_link_2"
+            reason="Adjacent" />
+        <disable_collisions link1="collision_head_link_1" link2="head" reason="Never" />
+        <disable_collisions link1="collision_head_link_1" link2="left_lower_shoulder" reason="Never" />
+        <disable_collisions link1="collision_head_link_1" link2="left_upper_elbow" reason="Never" />
+        <disable_collisions link1="collision_head_link_1" link2="left_upper_shoulder" reason="Never" />
+        <disable_collisions link1="collision_head_link_1" link2="pedestal" reason="Never" />
+        <disable_collisions link1="collision_head_link_1" link2="right_upper_elbow_visual"
+            reason="Never" />
+        <disable_collisions link1="collision_head_link_1" link2="right_lower_shoulder"
+            reason="Never" />
+        <disable_collisions link1="collision_head_link_1" link2="right_upper_shoulder"
+            reason="Never" />
+        <disable_collisions link1="collision_head_link_1" link2="screen" reason="Never" />
+        <disable_collisions link1="collision_head_link_1" link2="sonar_ring" reason="Never" />
+        <disable_collisions link1="collision_head_link_1" link2="torso" reason="Adjacent" />
+        <disable_collisions link1="collision_head_link_1" link2="display" reason="Adjacent" />
+        <disable_collisions link1="collision_head_link_2" link2="head" reason="Never" />
+        <disable_collisions link1="collision_head_link_2" link2="left_upper_shoulder" reason="Never" />
+        <disable_collisions link1="collision_head_link_2" link2="pedestal" reason="Never" />
+        <disable_collisions link1="collision_head_link_2" link2="right_lower_shoulder"
+            reason="Never" />
+        <disable_collisions link1="collision_head_link_2" link2="right_upper_elbow" reason="Never" />
+        <disable_collisions link1="collision_head_link_2" link2="right_upper_shoulder"
+            reason="Never" />
+        <disable_collisions link1="collision_head_link_2" link2="screen" reason="Never" />
+        <disable_collisions link1="collision_head_link_2" link2="sonar_ring" reason="Never" />
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