Commit message: update arm transfer

File: src/rethink_ee_description/urdf/electric_gripper/rethink_electric_gripper.xacro (robot description, xacro)
@@ -71,5 +71,5 @@
       <parent link="${side}_gripper_base" />
       <child link="${gripper_side}_gripper_l_finger" />
-      <limit effort="20.0" lower="0.0" upper="0.020833" velocity="5.0" />
+      <limit effort="200.0" lower="0.0" upper="0.020833" velocity="5.0" />
       <dynamics damping="0.7" friction="0.0" />
     </joint>
@@ -82,5 +82,5 @@
       <parent link="${side}_gripper_base" />
       <child link="${gripper_side}_gripper_r_finger" />
-      <limit effort="20.0" lower="-0.020833" upper="0.0" velocity="5.0" />
+      <limit effort="200.0" lower="-0.020833" upper="0.0" velocity="5.0" />
       <!-- <mimic joint="${gripper_side}_gripper_l_finger_joint" multiplier="-1.0" /> -->
       <dynamics damping="0.7" friction="0.0" />

File: src/webots_baxter/resource/kinect/urdf/kinect.urdf.xacro (robot description, xacro)
@@ -33,5 +33,5 @@
       <origin xyz=" 0 0 0 " rpy="0 0 0" />
       <geometry>
-        <mesh filename="package://webots_baxter/resource/kinect/meshes/kinect.dae"/>
+        <!-- <mesh filename="package://webots_baxter/resource/kinect/meshes/kinect.dae"/> -->
       </geometry>
     </visual>
